File: Controller/_autosave-Controller.kicad_sch (KiCad schematic)
At the start: 96 parts, among them J1 AudioJack3_SwitchTR, J10 AudioJack3_SwitchTR, J11 AudioJack3_SwitchTR, J12 AudioJack3_SwitchTR, J13 AudioJack3_SwitchTR, J14 AudioJack3_SwitchTR, J15 AudioJack3_SwitchTR, J16 EXT MODULE, J17 EXT MODULE, J18 AudioJack3_SwitchTR, J19 AudioJack3_SwitchTR, J2 AudioJack3_SwitchTR, J20 AudioJack3_SwitchTR, J21 AudioJack3_SwitchTR, J22 AudioJack3_SwitchTR, J23 AudioJack3_SwitchTR, J24 AudioJack3_SwitchTR, J25 AudioJack3_SwitchTR, J26 AudioJack3_SwitchTR, J27 AudioJack3_SwitchTR, J28 AudioJack3_SwitchTR, J29 AudioJack3_SwitchTR, J3 EURO_CONN, J30 AudioJack3_SwitchTR, J31 AudioJack3_SwitchTR, J32 AudioJack3_SwitchTR, J33 AudioJack3_SwitchTR, J34 AudioJack3_SwitchTR, J35 AudioJack3_SwitchTR, J36 AudioJack3_SwitchTR, J37 AudioJack3_SwitchTR, J38 AudioJack3_SwitchTR, J39 AudioJack3_SwitchTR, J4 AudioJack3_SwitchTR, J40 AudioJack3_SwitchTR, J41 AudioJack3_SwitchTR, J42 AudioJack3_SwitchTR, J43 AudioJack3_SwitchTR, J44 AudioJack3_SwitchTR, J45 AudioJack3_SwitchTR, J46 AudioJack3_SwitchTR, J5 AudioJack3_SwitchTR, J6 AudioJack3_SwitchTR, J7 AudioJack3_SwitchTR, J8 AudioJack3_SwitchTR, J9 AudioJack3_SwitchTR, SW1 XCHAN, SW2 DO MATH, SW3 SW_SPDT, SW4 SW_SPDT, U1 TL074, U2 TL074, U3 SN74HC32PWR, U4 SN74HC32PWR

Commit message: GET IT IN GITHUB NAO!
Parts:
- added J47, J48, J49, J50, J51, J52, J53, J54, J55, J56, J57, J58: AudioJack3_SwitchTR, AT-Footprints:CONN5_STX-3680_KYC, symbol Connector_Audio:AudioJack3_SwitchTR
Connections:
- net +5V: now also U4.14 (VCC)
- net GND: now also U4.7 (GND), J47.S, J48.S, J49.S, J50.S, J51.S, J52.S, J53.S, J54.S, J55.S, J56.S, J57.S, J58.S
- net at U4.1 (1A): now also J48.T
- net at U4.10 (3B): now also J50.T
- net at U4.11 (4Y): now also J58.T
- net at U4.12 (4A): now also J53.T
- net at U4.13 (4B): now also J56.T
- net at U4.2 (1B): now also J51.T
- net at U4.3 (1Y): now also J49.T
- net at U4.4 (2A): now also J54.T
- net at U4.5 (2B): now also J57.T
- net at U4.6 (2Y): now also J52.T
- net at U4.8 (3Y): now also J55.T
- net at U4.9 (3A): now also J47.T
- no-connect marks 42 -> 78
Other:
- moved on the sheet: J2, J35, J36, J37, J38, J39, J40, J41, J42, J43, J44, J45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
