File: Controller/Controller.kicad_pcb (KiCad board)
At the start: 2 copper layers, 99.5 x 101.5 mm, 54 parts, among them J1 Bus_EURO_Express, J1 EURO_EXPRESS, J2 10025026-10103TLF, J3 EURO_CONN, J5 ATX_POWER, J6 FRONT_PANEL, SW1 CH559_PRG, U1 DKA30A-12, U2 MAX16054, U4 TMUX4051PWR, U5 U_RP2040, U6 W25Q32JVSS, X1 12MHz

Commit message: i did a thing
Parts:
- removed the H5 at (90.8, 141.5)
- removed the H5 at (144.5, 52.3)
- removed the H6 at (231.9, 52.3)
- removed the H6 at (98.8, 141.5)
- removed the H7 at (108.1, 148.9)
- removed the H7 at (144.5, 125.3)
- removed H8: H_HOLE, llama_shared:H_ATX_PERF
- removed the J1 at (146.7, 136.3)
- removed the J1 at (102.7, 116.7)
- removed J2 (x2): 10025026-10103TLF, AT-Footprints:AMPHENOL_10025026-10103TLF
- removed SW1: CH559_PRG, llama_shared:SW_B3FS-1010
- removed U4: TMUX4051PWR, AT-Footprints:TSSOP16_PW_TEX
- removed U5: U_RP2040, llama_shared:U_QFN40P700X700X90-57N
- removed X1: 12MHz, llama_shared:X_SMD3225
- added C21: 2n2, Capacitor_SMD:C_0805_2012Metric_Pad1.18x1.45mm_HandSolder, F.Cu at (283.7, 86.4)
- added C22: 2n2, Capacitor_SMD:C_0805_2012Metric_Pad1.18x1.45mm_HandSolder, F.Cu at (283.7, 89.4)
- added C23: 1uF, Capacitor_SMD:C_0805_2012Metric_Pad1.18x1.45mm_HandSolder, F.Cu at (283.7, 92.4)
- added C24: 2n2, Capacitor_SMD:C_0805_2012Metric_Pad1.18x1.45mm_HandSolder, F.Cu at (288.5, 77.3)
- added C25: 1uF, Capacitor_SMD:C_0805_2012Metric_Pad1.18x1.45mm_HandSolder, F.Cu at (288.5, 80.3)
- added C26: 100nF, Capacitor_SMD:C_0805_2012Metric_Pad1.18x1.45mm_HandSolder, F.Cu at (288.5, 83.3)
- added C27: 100nF, Capacitor_SMD:C_0805_2012Metric_Pad1.18x1.45mm_HandSolder, F.Cu at (288.5, 86.4)
- added D1: 5V OK, LED_SMD:LED_0805_2012Metric, F.Cu at (114.8, 62.0)
- added D2: 12V OK, LED_SMD:LED_0805_2012Metric, F.Cu at (114.8, 65.0)
- added D3: -12V OK, LED_SMD:LED_0805_2012Metric, F.Cu at (114.8, 68.0)
- added D4: PWR_CONN, LED_SMD:LED_0805_2012Metric, F.Cu at (114.8, 71.0)
- added D5: 1N4148W, Diode_SMD:D_SOD-123, F.Cu at (286.8, 104.2)
- added D6: 1N4148W, Diode_SMD:D_SOD-123, F.Cu at (286.8, 107.5)
- added G***: LOGO, AT-Footprints:gfx_ehlo_backgr, F.Cu at (117.8, 134.9)
- added H2: MountingHole, MountingHole:MountingHole_3.2mm_M3, F.Cu at (121.0, 64.4)
- added H5: H_HOLE, llama_shared:H_ATX_PERF, F.Cu at (101.4, 72.5)
- added H6: H_HOLE, llama_shared:H_ATX_PERF, F.Cu at (101.4, 80.5)
- added H7: H_HOLE, llama_shared:H_ATX_PERF, F.Cu at (101.4, 88.5)
- added J1: AudioJack3_SwitchTR, AT-Footprints:CONN5_STX-3680_KYC, F.Cu at (71.5, 56.5)
- added J4: AudioJack3_SwitchTR, AT-Footprints:CONN5_STX-3680_KYC, F.Cu at (84.0, 56.5)
- added J7: AudioJack3_SwitchTR, AT-Footprints:CONN5_STX-3680_KYC, F.Cu at (121.5, 56.5)
- added J87: AudioJack3_SwitchTR, AT-Footprints:CONN5_STX-3680_KYC, F.Cu at (213.8, 36.5)
- added J88: AudioJack3_SwitchTR, AT-Footprints:CONN5_STX-3680_KYC, F.Cu at (226.3, 36.5)
- added J89: AudioJack3_SwitchTR, AT-Footprints:CONN5_STX-3680_KYC, F.Cu at (238.8, 36.5)
- added J90: AudioJack3_SwitchTR, AT-Footprints:CONN5_STX-3680_KYC, F.Cu at (251.3, 36.5)
- added Q1: BC548, Package_TO_SOT_THT:TO-92_Inline, F.Cu at (254.2, 79.1)
- added Q10: BC548, Package_TO_SOT_THT:TO-92_Inline, F.Cu at (260.7, 96.5)
- added Q11: BC548, Package_TO_SOT_THT:TO-92_Inline, F.Cu at (260.7, 102.2)
- added Q12: BC548, Package_TO_SOT_THT:TO-92_Inline, F.Cu at (260.7, 108.0)
- added Q13: BC548, Package_TO_SOT_THT:TO-92_Inline, F.Cu at (267.2, 79.1)
- added Q14: BC558, Package_TO_SOT_THT:TO-92_Inline, F.Cu at (267.2, 84.9)
- added Q15: BC558, Package_TO_SOT_THT:TO-92_Inline, F.Cu at (267.2, 90.7)
- added Q16: BC548, Package_TO_SOT_THT:TO-92_Inline, F.Cu at (267.2, 96.5)
- added Q17: BC548, Package_TO_SOT_THT:TO-92_Inline, F.Cu at (267.2, 102.2)
- added Q18: BC548, Package_TO_SOT_THT:TO-92_Inline, F.Cu at (267.2, 108.0)
- added Q2: BC558, Package_TO_SOT_THT:TO-92_Inline, F.Cu at (254.2, 84.9)
- added Q3: BC558, Package_TO_SOT_THT:TO-92_Inline, F.Cu at (254.2, 90.7)
- added Q4: BC548, Package_TO_SOT_THT:TO-92_Inline, F.Cu at (254.2, 96.5)
- added Q5: BC558, Package_TO_SOT_THT:TO-92_Inline, F.Cu at (254.2, 102.2)
- added Q6: BC548, Package_TO_SOT_THT:TO-92_Inline, F.Cu at (254.2, 108.0)
- added Q7: BC558, Package_TO_SOT_THT:TO-92_Inline, F.Cu at (260.7, 79.1)
- added Q8: BC548, Package_TO_SOT_THT:TO-92_Inline, F.Cu at (260.7, 84.9)
- added Q9: BC548, Package_TO_SOT_THT:TO-92_Inline, F.Cu at (260.7, 90.7)
- added R13: 10k 0.1%, Resistor_SMD:R_0805_2012Metric_Pad1.20x1.40mm_HandSolder, B.Cu at (146.8, 93.9)
- added R137: 100k, Resistor_SMD:R_0805_2012Metric_Pad1.20x1.40mm_HandSolder, F.Cu at (273.6, 62.5)
- added R138: 33k, Resistor_SMD:R_0805_2012Metric_Pad1.20x1.40mm_HandSolder, F.Cu at (273.6, 65.5)
- added R139: 100k, Resistor_SMD:R_0805_2012Metric_Pad1.20x1.40mm_HandSolder, F.Cu at (273.6, 68.5)
- added R14: 1k 0.1%, Resistor_SMD:R_0805_2012Metric_Pad1.20x1.40mm_HandSolder, F.Cu at (150.8, 94.7)
- added R140: 100k, Resistor_SMD:R_0805_2012Metric_Pad1.20x1.40mm_HandSolder, F.Cu at (273.6, 71.4)
- added R141: 1k5, Resistor_SMD:R_0805_2012Metric_Pad1.20x1.40mm_HandSolder, F.Cu at (273.6, 74.3)
- added R142: 100k, Resistor_SMD:R_0805_2012Metric_Pad1.20x1.40mm_HandSolder, F.Cu at (278.3, 41.9)
- added R143: 1M, Resistor_SMD:R_0805_2012Metric_Pad1.20x1.40mm_HandSolder, F.Cu at (278.3, 44.9)
- added R144: 100k, Resistor_SMD:R_0805_2012Metric_Pad1.20x1.40mm_HandSolder, F.Cu at (278.3, 47.8)
- added R145: 1M, Resistor_SMD:R_0805_2012Metric_Pad1.20x1.40mm_HandSolder, F.Cu at (278.3, 50.8)
- added R146: 100k, Resistor_SMD:R_0805_2012Metric_Pad1.20x1.40mm_HandSolder, F.Cu at (278.3, 53.7)
- added R147: 68k, Resistor_SMD:R_0805_2012Metric_Pad1.20x1.40mm_HandSolder, F.Cu at (278.3, 56.6)
- added R148: 100k, Resistor_SMD:R_0805_2012Metric_Pad1.20x1.40mm_HandSolder, F.Cu at (278.3, 59.6)
- added R149: 14k, Resistor_SMD:R_0805_2012Metric_Pad1.20x1.40mm_HandSolder, F.Cu at (278.3, 62.5)
- added R15: 10k 0.1%, Resistor_SMD:R_0805_2012Metric_Pad1.20x1.40mm_HandSolder, F.Cu at (117.2, 84.3)
- added R150: 47k, Resistor_SMD:R_0805_2012Metric_Pad1.20x1.40mm_HandSolder, F.Cu at (278.3, 65.5)
- added R151: 100k, Resistor_SMD:R_0805_2012Metric_Pad1.20x1.40mm_HandSolder, F.Cu at (278.3, 68.5)
- added R152: 68k, Resistor_SMD:R_0805_2012Metric_Pad1.20x1.40mm_HandSolder, F.Cu at (278.3, 71.4)
- added R153: 100k, Resistor_SMD:R_0805_2012Metric_Pad1.20x1.40mm_HandSolder, F.Cu at (278.3, 74.3)
- added R154: 1k, Resistor_SMD:R_0805_2012Metric_Pad1.20x1.40mm_HandSolder, F.Cu at (283.1, 41.9)
- added R155: 1k, Resistor_SMD:R_0805_2012Metric_Pad1.20x1.40mm_HandSolder, F.Cu at (283.1, 44.9)
- added R156: 10k, Resistor_SMD:R_0805_2012Metric_Pad1.20x1.40mm_HandSolder, F.Cu at (283.1, 47.8)
- added R157: 10k, Resistor_SMD:R_0805_2012Metric_Pad1.20x1.40mm_HandSolder, F.Cu at (283.1, 50.8)
- added R158: 1k, Resistor_SMD:R_0805_2012Metric_Pad1.20x1.40mm_HandSolder, F.Cu at (283.1, 53.7)
- added R159: 100k, Resistor_SMD:R_0805_2012Metric_Pad1.20x1.40mm_HandSolder, F.Cu at (283.1, 56.6)
- added R16: 10k 0.1%, Resistor_SMD:R_0805_2012Metric_Pad1.20x1.40mm_HandSolder, F.Cu at (117.2, 87.3)
- added R160: 100k, Resistor_SMD:R_0805_2012Metric_Pad1.20x1.40mm_HandSolder, F.Cu at (283.1, 59.6)
- added R161: 100k, Resistor_SMD:R_0805_2012Metric_Pad1.20x1.40mm_HandSolder, F.Cu at (283.1, 62.5)
- added R162: 1k, Resistor_SMD:R_0805_2012Metric_Pad1.20x1.40mm_HandSolder, F.Cu at (283.1, 65.5)
- added R17: 10k 0.1%, Resistor_SMD:R_0805_2012Metric_Pad1.20x1.40mm_HandSolder, F.Cu at (117.2, 90.2)
- added R18: 51k, Resistor_SMD:R_0805_2012Metric_Pad1.20x1.40mm_HandSolder, F.Cu at (254.6, 41.9)
- added R19: 1k, Resistor_SMD:R_0805_2012Metric_Pad1.20x1.40mm_HandSolder, F.Cu at (254.6, 44.9)
- added R20: 10k, Resistor_SMD:R_0805_2012Metric_Pad1.20x1.40mm_HandSolder, F.Cu at (254.6, 47.8)
- added R21: 20k, Resistor_SMD:R_0805_2012Metric_Pad1.20x1.40mm_HandSolder, F.Cu at (254.6, 50.8)
- added R22: 10k 0.1%, Resistor_SMD:R_0805_2012Metric_Pad1.20x1.40mm_HandSolder, F.Cu at (117.2, 93.2)
- added R23: 1k 0.1%, Resistor_SMD:R_0805_2012Metric_Pad1.20x1.40mm_HandSolder, F.Cu at (117.2, 96.1)
- added R24: 1k 0.1%, Resistor_SMD:R_0805_2012Metric_Pad1.20x1.40mm_HandSolder, F.Cu at (117.2, 99.1)
- added R25: 10k 0.1%, Resistor_SMD:R_0805_2012Metric_Pad1.20x1.40mm_HandSolder, F.Cu at (117.2, 102.0)
- added R26: 10k 0.1%, Resistor_SMD:R_0805_2012Metric_Pad1.20x1.40mm_HandSolder, F.Cu at (122.0, 84.3)
- added R27: 10k 0.1%, Resistor_SMD:R_0805_2012Metric_Pad1.20x1.40mm_HandSolder, F.Cu at (122.0, 87.3)
- added R28: 10k 0.1%, Resistor_SMD:R_0805_2012Metric_Pad1.20x1.40mm_HandSolder, F.Cu at (122.0, 90.2)
- added R29: 1k 0.1%, Resistor_SMD:R_0805_2012Metric_Pad1.20x1.40mm_HandSolder, F.Cu at (122.0, 93.2)
- added R30: 1k 0.1%, Resistor_SMD:R_0805_2012Metric_Pad1.20x1.40mm_HandSolder, F.Cu at (122.0, 96.1)
- added R31: 20k, Resistor_SMD:R_0805_2012Metric_Pad1.20x1.40mm_HandSolder, F.Cu at (254.6, 53.7)
- added R32: 20k, Resistor_SMD:R_0805_2012Metric_Pad1.20x1.40mm_HandSolder, F.Cu at (254.6, 56.6)
- added R33: 20k, Resistor_SMD:R_0805_2012Metric_Pad1.20x1.40mm_HandSolder, F.Cu at (254.6, 59.6)
- added R34: 20k, Resistor_SMD:R_0805_2012Metric_Pad1.20x1.40mm_HandSolder, F.Cu at (254.6, 62.5)
- added R35: 10k, Resistor_SMD:R_0805_2012Metric_Pad1.20x1.40mm_HandSolder, F.Cu at (254.6, 65.5)
- added R36: 200k, Resistor_SMD:R_0805_2012Metric_Pad1.20x1.40mm_HandSolder, F.Cu at (254.6, 68.5)
- added R37: 1k, Resistor_SMD:R_0805_2012Metric_Pad1.20x1.40mm_HandSolder, F.Cu at (254.6, 71.4)
- added R38: 51k, Resistor_SMD:R_0805_2012Metric_Pad1.20x1.40mm_HandSolder, F.Cu at (254.6, 74.3)
- added R39: 1k, Resistor_SMD:R_0805_2012Metric_Pad1.20x1.40mm_HandSolder, F.Cu at (259.3, 41.9)
- added R40: 20k, Resistor_SMD:R_0805_2012Metric_Pad1.20x1.40mm_HandSolder, F.Cu at (259.3, 44.9)
- added R41: 20k, Resistor_SMD:R_0805_2012Metric_Pad1.20x1.40mm_HandSolder, F.Cu at (259.3, 47.8)
- added R42: 10k, Resistor_SMD:R_0805_2012Metric_Pad1.20x1.40mm_HandSolder, F.Cu at (259.3, 50.8)
- added R43: 20k, Resistor_SMD:R_0805_2012Metric_Pad1.20x1.40mm_HandSolder, F.Cu at (259.3, 53.7)
- added R44: 20k, Resistor_SMD:R_0805_2012Metric_Pad1.20x1.40mm_HandSolder, F.Cu at (259.3, 56.6)
- added R45: 20k, Resistor_SMD:R_0805_2012Metric_Pad1.20x1.40mm_HandSolder, F.Cu at (259.3, 59.6)
- added R46: 10k, Resistor_SMD:R_0805_2012Metric_Pad1.20x1.40mm_HandSolder, F.Cu at (259.3, 62.5)
- added R47: 200k, Resistor_SMD:R_0805_2012Metric_Pad1.20x1.40mm_HandSolder, F.Cu at (259.3, 65.5)
- added R48: 1k, Resistor_SMD:R_0805_2012Metric_Pad1.20x1.40mm_HandSolder, F.Cu at (259.3, 68.5)
- added R49: 10k, Resistor_SMD:R_0805_2012Metric_Pad1.20x1.40mm_HandSolder, F.Cu at (259.3, 71.4)
- added R50: 10k, Resistor_SMD:R_0805_2012Metric_Pad1.20x1.40mm_HandSolder, F.Cu at (259.3, 74.3)
- added R51: 1k, Resistor_SMD:R_0805_2012Metric_Pad1.20x1.40mm_HandSolder, F.Cu at (264.1, 41.9)
- added R52: 100k, Resistor_SMD:R_0805_2012Metric_Pad1.20x1.40mm_HandSolder, F.Cu at (264.1, 44.9)
- added R53: 100k, Resistor_SMD:R_0805_2012Metric_Pad1.20x1.40mm_HandSolder, F.Cu at (264.1, 47.8)
- added R54: 100k, Resistor_SMD:R_0805_2012Metric_Pad1.20x1.40mm_HandSolder, F.Cu at (264.1, 50.8)
- added R55: 1k, Resistor_SMD:R_0805_2012Metric_Pad1.20x1.40mm_HandSolder, F.Cu at (264.1, 53.7)
- added R56: 10k, Resistor_SMD:R_0805_2012Metric_Pad1.20x1.40mm_HandSolder, F.Cu at (264.1, 56.6)
- added R57: 10k, Resistor_SMD:R_0805_2012Metric_Pad1.20x1.40mm_HandSolder, F.Cu at (264.1, 59.6)
- added R58: 1k, Resistor_SMD:R_0805_2012Metric_Pad1.20x1.40mm_HandSolder, F.Cu at (264.1, 62.5)
- added R59: 100k, Resistor_SMD:R_0805_2012Metric_Pad1.20x1.40mm_HandSolder, F.Cu at (264.1, 65.5)
- added R60: 100k, Resistor_SMD:R_0805_2012Metric_Pad1.20x1.40mm_HandSolder, F.Cu at (264.1, 68.5)
- added R61: 100k, Resistor_SMD:R_0805_2012Metric_Pad1.20x1.40mm_HandSolder, F.Cu at (264.1, 71.4)
- added R62: 1k, Resistor_SMD:R_0805_2012Metric_Pad1.20x1.40mm_HandSolder, F.Cu at (264.1, 74.3)
- added R63: 47k, Resistor_SMD:R_0805_2012Metric_Pad1.20x1.40mm_HandSolder, F.Cu at (268.8, 41.9)
- added R64: 100k, Resistor_SMD:R_0805_2012Metric_Pad1.20x1.40mm_HandSolder, F.Cu at (268.8, 44.9)
- added R65: 1k, Resistor_SMD:R_0805_2012Metric_Pad1.20x1.40mm_HandSolder, F.Cu at (268.8, 47.8)
- added R66: 1k, Resistor_SMD:R_0805_2012Metric_Pad1.20x1.40mm_HandSolder, F.Cu at (268.8, 50.8)
- added R67: 100k, Resistor_SMD:R_0805_2012Metric_Pad1.20x1.40mm_HandSolder, F.Cu at (268.8, 53.7)
- added R68: 68k, Resistor_SMD:R_0805_2012Metric_Pad1.20x1.40mm_HandSolder, F.Cu at (268.8, 56.6)
- added R69: 14k, Resistor_SMD:R_0805_2012Metric_Pad1.20x1.40mm_HandSolder, F.Cu at (268.8, 59.6)
- added R70: 68k, Resistor_SMD:R_0805_2012Metric_Pad1.20x1.40mm_HandSolder, F.Cu at (268.8, 62.5)
- added R71: 100k, Resistor_SMD:R_0805_2012Metric_Pad1.20x1.40mm_HandSolder, F.Cu at (268.8, 65.5)
- added R72: 100k, Resistor_SMD:R_0805_2012Metric_Pad1.20x1.40mm_HandSolder, F.Cu at (268.8, 68.5)
- added R73: 1M, Resistor_SMD:R_0805_2012Metric_Pad1.20x1.40mm_HandSolder, F.Cu at (268.8, 71.4)
- added R74: 1k5, Resistor_SMD:R_0805_2012Metric_Pad1.20x1.40mm_HandSolder, F.Cu at (268.8, 74.3)
- added R75: 100k, Resistor_SMD:R_0805_2012Metric_Pad1.20x1.40mm_HandSolder, F.Cu at (273.6, 41.9)
- added R76: 100k, Resistor_SMD:R_0805_2012Metric_Pad1.20x1.40mm_HandSolder, F.Cu at (273.6, 44.9)
- added R77: 33k, Resistor_SMD:R_0805_2012Metric_Pad1.20x1.40mm_HandSolder, F.Cu at (273.6, 47.8)
- added R78: 100k, Resistor_SMD:R_0805_2012Metric_Pad1.20x1.40mm_HandSolder, F.Cu at (273.6, 50.8)
- added R79: 100k, Resistor_SMD:R_0805_2012Metric_Pad1.20x1.40mm_HandSolder, F.Cu at (273.6, 53.7)
- added R80: 1M, Resistor_SMD:R_0805_2012Metric_Pad1.20x1.40mm_HandSolder, F.Cu at (273.6, 56.6)
- added R81: 100k, Resistor_SMD:R_0805_2012Metric_Pad1.20x1.40mm_HandSolder, F.Cu at (273.6, 59.6)
- added RV10: 10k, Potentiometer_THT:Potentiometer_Bourns_PTV09A-1_Single_Vertical, F.Cu at (207.5, 78.8)
- added RV11: 250k, Potentiometer_THT:Potentiometer_Bourns_PTV09A-1_Single_Vertical, F.Cu at (207.5, 93.2)
- added RV12: 100k, Potentiometer_THT:Potentiometer_Runtron_RM-065_Vertical, F.Cu at (273.3, 96.0)
- added RV13: 100k, Potentiometer_THT:Potentiometer_Bourns_PTV09A-1_Single_Vertical, F.Cu at (207.5, 107.5)
- added RV14: 100k, Potentiometer_THT:Potentiometer_Bourns_PTV09A-1_Single_Vertical, F.Cu at (223.0, 50.1)
- added RV15: 100k, Potentiometer_THT:Potentiometer_Bourns_PTV09A-1_Single_Vertical, F.Cu at (223.0, 64.5)
- added RV16: 100k, Potentiometer_THT:Potentiometer_Bourns_PTV09A-1_Single_Vertical, F.Cu at (223.0, 78.8)
- added RV17: 100k, Potentiometer_THT:Potentiometer_Bourns_PTV09A-1_Single_Vertical, F.Cu at (223.0, 93.2)
- added RV18: 100k, Potentiometer_THT:Potentiometer_Bourns_PTV09A-1_Single_Vertical, F.Cu at (223.0, 107.5)
- added RV19: 100k, Potentiometer_THT:Potentiometer_Runtron_RM-065_Vertical, F.Cu at (281.4, 96.0)
- added RV20: 100k, Potentiometer_THT:Potentiometer_Bourns_PTV09A-1_Single_Vertical, F.Cu at (238.4, 50.1)
- added RV21: 100k, Potentiometer_THT:Potentiometer_Bourns_PTV09A-1_Single_Vertical, F.Cu at (238.4, 64.5)
- added RV22: 250k, Potentiometer_THT:Potentiometer_Bourns_PTV09A-1_Single_Vertical, F.Cu at (238.4, 78.8)
- added RV23: 10k, Potentiometer_THT:Potentiometer_Bourns_PTV09A-1_Single_Vertical, F.Cu at (238.4, 93.2)
- added RV7: 10k, Potentiometer_THT:Potentiometer_Bourns_PTV09A-1_Single_Vertical, F.Cu at (-135.6, 87.5)
- added RV8: 10k, Potentiometer_THT:Potentiometer_Bourns_PTV09A-1_Single_Vertical, F.Cu at (207.5, 50.1)
- added RV9: 10k, Potentiometer_THT:Potentiometer_Bourns_PTV09A-1_Single_Vertical, F.Cu at (207.5, 64.5)
- added TP1: C, TestPoint:TestPoint_Pad_1.0x1.0mm, F.Cu at (273.2, 104.0)
- added TP2: D, TestPoint:TestPoint_Pad_1.0x1.0mm, F.Cu at (273.2, 107.1)
- added TP3: B, TestPoint:TestPoint_Pad_1.0x1.0mm, F.Cu at (276.3, 104.0)
- added TP4: A, TestPoint:TestPoint_Pad_1.0x1.0mm, F.Cu at (276.3, 107.1)
- added TP5: A, TestPoint:TestPoint_Pad_1.0x1.0mm, F.Cu at (279.3, 104.0)
- added TP6: B, TestPoint:TestPoint_Pad_1.0x1.0mm, F.Cu at (279.3, 107.1)
- added TP7: D, TestPoint:TestPoint_Pad_1.0x1.0mm, F.Cu at (282.4, 104.0)
- added TP8: C, TestPoint:TestPoint_Pad_1.0x1.0mm, F.Cu at (282.4, 107.1)
- added U10: TL074, AT-Footprints:SOT23_DYY_TEX, F.Cu at (288.2, 61.7)
- added U13: TL074, AT-Footprints:SOT23_DYY_TEX, F.Cu at (288.2, 67.6)
- added U7: TL072, Package_SO:TSSOP-8_4.4x3mm_P0.65mm, F.Cu at (289.8, 47.3)
- added U8: TL072, Package_SO:TSSOP-8_4.4x3mm_P0.65mm, F.Cu at (289.8, 51.9)
- added U9: TL072, Package_SO:TSSOP-8_4.4x3mm_P0.65mm, F.Cu at (289.8, 56.5)
- C1: value 0.1uF -> 10pF; moved to F.Cu
- C10, C11, C12, C13, C14, C15: value 0.1uF -> 100nF; footprint llama_shared:C_0402_1005Metric -> Capacitor_SMD:C_0805_2012Metric_Pad1.18x1.45mm_HandSolder
- C16, C17: value 1uF -> 100nF; footprint llama_shared:C_0402_1005Metric -> Capacitor_SMD:C_0805_2012Metric_Pad1.18x1.45mm_HandSolder
- C18, C19: value 30pF -> 100nF; footprint llama_shared:C_0402_1005Metric -> Capacitor_SMD:C_0805_2012Metric_Pad1.18x1.45mm_HandSolder
- C2: value 10uF -> 100nF
- C20, C9: value 0.1uF -> 1uF; footprint llama_shared:C_0402_1005Metric -> Capacitor_SMD:C_0805_2012Metric_Pad1.18x1.45mm_HandSolder
- C3, C4, C5: value 100uF -> 100nF; footprint llama_shared:C_1210_3225Metric -> Capacitor_SMD:C_0805_2012Metric_Pad1.18x1.45mm_HandSolder
- C6: value 100uF -> 1uF; footprint llama_shared:C_1210_3225Metric -> Capacitor_SMD:C_0805_2012Metric_Pad1.18x1.45mm_HandSolder
- C7, C8: value 0.1uF -> 2n2; footprint llama_shared:C_0402_1005Metric -> Capacitor_SMD:C_0805_2012Metric_Pad1.18x1.45mm_HandSolder
- J3: footprint AT-Footprints:EURORACK Right Angle -> Connector_PinHeader_2.54mm:PinHeader_2x08_P2.54mm_Vertical
- J5: value ATX_POWER -> AudioJack3_SwitchTR; footprint ATX:ATX_24_RIGHT_ANGLE_MOLEX_469911024 -> AT-Footprints:CONN5_STX-3680_KYC
- J6: value FRONT_PANEL -> AudioJack3_SwitchTR; footprint llama_shared:P_CONN_PANEL -> AT-Footprints:CONN5_STX-3680_KYC
- R1: value 10k -> 100k 0.1%
- R10: value 1k -> 150; footprint llama_shared:R_0402_1005Metric -> Resistor_SMD:R_0805_2012Metric_Pad1.20x1.40mm_HandSolder
- R11: value 10k -> 500; footprint llama_shared:R_0402_1005Metric -> Resistor_SMD:R_0805_2012Metric_Pad1.20x1.40mm_HandSolder
- R12: value 1k -> 500; footprint llama_shared:R_0402_1005Metric -> Resistor_SMD:R_0805_2012Metric_Pad1.20x1.40mm_HandSolder
- R2: value 470 -> 100k 0.1%; moved to F.Cu
- R3: value 330 -> 100k 0.1%; moved to B.Cu
- R4: value 470 -> 100k 0.1%
- R5: value 470 -> 10k 0.1%; moved to F.Cu
- R6: value 470 -> 10k 0.1%
- R7: value 470 -> 1k 0.1%; moved to F.Cu
- R8: value 330 -> 10k 0.1%; moved to F.Cu
- R9: value 10k -> 150; footprint llama_shared:R_0402_1005Metric -> Resistor_SMD:R_0805_2012Metric_Pad1.20x1.40mm_HandSolder
- U1: value DKA30A-12 -> TL074; footprint AT-Footprints:DKA30_MWU -> AT-Footprints:SOT23_DYY_TEX
- U2: value MAX16054 -> TL074; footprint llama_shared:U_TSOT-23-6 -> AT-Footprints:SOT23_DYY_TEX
- U6: value W25Q32JVSS -> TL072; footprint llama_shared:U_SOIC-8_5.23x5.23mm_P1.27mm -> Package_SO:TSSOP-8_4.4x3mm_P0.65mm
- moved R9 161.9 mm to (112.5, 87.3)
- moved R10 161.5 mm to (112.5, 90.2)
- moved R11 161.2 mm to (112.5, 93.2)
- moved R12 160.8 mm to (112.5, 96.1)
- moved R1 114.2 mm to (107.7, 84.3), turned to 0 degrees
- moved R2 113.2 mm to (107.7, 87.3), turned to 0 degrees
- moved J6 111.7 mm to (109.0, 56.5), turned to 0 degrees
- moved R4 98.2 mm to (140.3, 99.4), turned to 0 degrees
- moved U6 93.6 mm to (289.8, 42.7)
- moved R5 93.5 mm to (146.8, 100.9), turned to 180 degrees
- moved J3 91.5 mm to (107.7, 62.8)
- moved R6 88.8 mm to (146.8, 100.9), turned to 0 degrees
- moved R3 86.1 mm to (142.8, 94.7), turned to -90 degrees
- moved R7 85.5 mm to (150.8, 100.2), turned to 90 degrees
- moved C1 83.8 mm to (142.8, 94.7), turned to 90 degrees
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Connections:
- C1 pad 1: GND -> Net-(U1A--)
- C1 pad 2: +5VSB -> /BMULT_L
- C10 pad 2: RP_3.3V -> +12V
- C11 pad 1: GND -> -12V
- C11 pad 2: RP_3.3V -> GND
- C12 pad 2: RP_3.3V -> +12V
- C13 pad 1: GND -> -12V
- C13 pad 2: RP_3.3V -> GND
- C14 pad 2: RP_1.1V -> +12V
- C15 pad 1: GND -> -12V
- C15 pad 2: RP_1.1V -> GND
- C16 pad 1: RP_3.3V -> GND
- C16 pad 2: GND -> +12V
- C17 pad 1: RP_1.1V -> -12V
- C18 pad 1: Net-(C18-Pad1) -> GND
- C18 pad 2: GND -> +12V
- C19 pad 1: Net-(U5-XIN) -> -12V
- C2 pad 1: /~{RST_SIG} -> GND
- C2 pad 2: GND -> +12V
- C20 pad 1: GND -> Net-(U10B-+)
- C20 pad 2: RP_3.3V -> Net-(U10A--)
- C3 pad 1: VCC -> -12V
- C4 pad 1: +12V -> GND
- C4 pad 2: GND -> +12V
- C5 pad 1: +3.3V -> -12V
- C6 pad 1: GND -> Net-(C6-Pad1)
- C6 pad 2: -12V -> Net-(C6-Pad2)
- C7 pad 2: RP_3.3V -> Net-(C6-Pad1)
- C8 pad 2: RP_3.3V -> Net-(C8-Pad2)
- C9 pad 1: GND -> Net-(C8-Pad2)
- C9 pad 2: RP_3.3V -> Net-(U9B-+)
- R1 pad 1: VCC -> Net-(U1A--)
- R1 pad 2: /~{RST_SW} -> Net-(J1-PadT)
- R10 pad 1: Net-(U5-XOUT) -> GND
- R10 pad 2: Net-(C18-Pad1) -> Net-(D1-K)
- R11 pad 1: /QSPI_CS -> GND
- R11 pad 2: RP_3.3V -> Net-(D2-K)
- R12 pad 1: /QSPI_CS -> Net-(D3-A)
- R12 pad 2: /BOOTSEL -> GND
- R2 pad 1: /~{RST_SIG} -> Net-(U1A--)
- R2 pad 2: /~{RST_SW} -> Net-(J4-PadT)
- R3 pad 1: VCC -> /BMULT_L
- R3 pad 2: /HDD_LED+ -> Net-(U1A--)
- R4 pad 1: +5VSB -> Net-(SW2-A)
- R4 pad 2: GND -> Net-(U1A--)
- R5 pad 1: VCC -> Net-(U1C--)
- R5 pad 2: GND -> unconnected-(R5-Pad2)
- R6 pad 1: +3.3V -> Net-(R6-Pad1)
- R6 pad 2: GND -> Net-(U1C--)
- R7 pad 1: +12V -> Net-(J5-PadR)
- R7 pad 2: GND -> Net-(R6-Pad1)
- R8 pad 1: VCC -> Net-(U1D--)
- R8 pad 2: /PWR_LED+ -> /BMULT_L
- R9 pad 1: unconnected-(R9-Pad1) -> GND
- U1 pad 1: unconnected-(U1-RC-Pad1) -> /BMULT_L
- U1 pad 5: +12VA -> unconnected-(U1B-+-Pad5)
- U1 pad 6: GNDA -> unconnected-(U1B---Pad6)
- U1 pad 7: -12VA -> unconnected-(U1-Pad7)
- U1 pad 8: unconnected-(U1-TRIM-Pad8) -> Net-(R6-Pad1)
- U2 pad 1: /~{PWR_SW} -> Net-(R27-Pad1)
- U2 pad 2: GND -> Net-(U2A--)
- U2 pad 4: /~{PS_ON} -> +12V
- U2 pad 5: unconnected-(U2-OUT-Pad5) -> GND
- U2 pad 6: +5VSB -> Net-(U2B--)
- U6 pad 1: /QSPI_CS -> Net-(Q1-B)
- U6 pad 2: /QSPI_SD1 -> Net-(Q1-B)
- U6 pad 3: /QSPI_SD2 -> Net-(U6A-+)
- U6 pad 4: GND -> -12V
- U6 pad 5: /QSPI_SD0 -> Net-(U6B-+)
- U6 pad 6: /QSPI_SCK -> Net-(Q5-B)
- U6 pad 7: /QSPI_SD3 -> Net-(Q5-B)
- U6 pad 8: RP_3.3V -> +12V
Routing:
- net +12V: track 103.9 -> 4.73 mm, vias 0 -> 2
- net +3.3V: track 69.5 -> 0.00 mm
- net VCC: track 68.8 -> 0.00 mm
- net +5VSB: track 61.1 -> 0.00 mm, vias 1 -> 0
- net /~{PS_ON}: track 28.8 -> 0.00 mm
- net -12V: track 16.1 -> 5.03 mm, vias 0 -> 2
- net /~{RST_SW}: track 10.9 -> 0.00 mm
- net /BMULT_L: track 0.00 -> 10.8 mm, vias 0 -> 1
- net /~{PWR_SW}: track 9.16 -> 0.00 mm
- net /PWR_LED-: track 7.73 -> 0.00 mm
- net Net-(U1D--): track 0.00 -> 5.72 mm, vias 0 -> 1
- net Net-(R13-Pad1): track 0.00 -> 5.49 mm, vias 0 -> 1
- net /HDD_LED+: track 5.04 -> 0.00 mm
- net GND: track 3.92 -> 0.00 mm
- net /HDD_LED-: track 3.90 -> 0.00 mm
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- removed copper zone on B.Cu, net GND
Other:
- board size 99.5 x 101.5 mm -> 100 x 100 mm
