File: Controller/Controller.kicad_sch (KiCad schematic)
At the start: 70 parts, among them J1 AudioJack3_SwitchTR, J16 EXT MODULE, J17 EXT MODULE, J2 USB_C_Receptacle_PowerOnly_6P, J3 EURO_CONN, J4 AudioJack3_SwitchTR, J5 AudioJack3_SwitchTR, J6 AudioJack3_SwitchTR, J7 AudioJack3_SwitchTR, Q2 2N3904, SW1 XCHAN, SW2 DO MATH, U1 TL074, U10 LM2596T-12, U2 TL074, U3 STUSB4500QTR, U9 LM2596T-12

Commit message: GET IT IN GITHUB NAO!
Parts:
- removed C14, C15: 680uF, Capacitor_SMD:C_0805_2012Metric_Pad1.18x1.45mm_HandSolder, symbol Device:C
- removed C16: 180uF, Capacitor_THT:CP_Radial_D10.0mm_P5.00mm, symbol Device:C
- removed D10: SMAZ18-13-F, Diode_SMD:D_SMA, symbol Diode:Z1SMAxxx
- removed D11: SK33, AT-Footprints:M-FLAT_TOS, symbol Device:D_Schottky
- removed D9: SK32, AT-Footprints:M-FLAT_TOS, symbol Device:D_Schottky
- removed HS1, HS5: HSE-B250-04H, AT-Footprints:HSINK_HSE-B250-04H, symbol AT-Symbols:HSE-B250-04H
- removed J2: USB_C_Receptacle_PowerOnly_6P, symbol Connector:USB_C_Receptacle_PowerOnly_6P
- removed L4: 53uH, AT-Footprints:IND_HCTI-68-7.7, symbol Device:L
- removed Q2: 2N3904, Package_TO_SOT_THT:TO-92_Inline, symbol Transistor_BJT:2N3904
- removed R18, R19: 10k, Resistor_SMD:R_0805_2012Metric_Pad1.20x1.40mm_HandSolder, symbol Device:R
- removed R20: 47k, Resistor_SMD:R_0805_2012Metric_Pad1.20x1.40mm_HandSolder, symbol Device:R
- removed R21: 1k, Resistor_SMD:R_0805_2012Metric_Pad1.20x1.40mm_HandSolder, symbol Device:R
- removed U10, U9: LM2596T-12, Package_TO_SOT_THT:TO-220-5_P3.4x3.7mm_StaggerOdd_Lead3.8mm_Vertical, symbol Regulator_Switching:LM2596T-12
- removed U3: STUSB4500QTR, Package_DFN_QFN:QFN-24-1EP_4x4mm_P0.5mm_EP2.7x2.7mm, symbol Interface_USB:STUSB4500QTR
- added J10, J11, J12, J13, J14, J15, J18, J19, J2, J20, J21, J22, J23, J24, J25, J26, J27, J28, J29, J30, J31, J32, J33, J34, J35, J36, J37, J38, J39, J40, J41, J42, J43, J44, J45, J46, J8, J9: AudioJack3_SwitchTR, AT-Footprints:CONN5_STX-3680_KYC, symbol Connector_Audio:AudioJack3_SwitchTR
- added RV1, RV2: R_Potentiometer, Potentiometer_THT:Potentiometer_Bourns_PTV09A-1_Single_Vertical, symbol Device:R_Potentiometer
- added SW3, SW4: SW_SPDT, symbol Switch:SW_SPDT
- added U3: SN74HC32PWR, Package_SO:TSSOP-14_4.4x5mm_P0.65mm, symbol AT-Symbols:SN74HC32PWR
- U1, U2: footprint (none) -> AT-Footprints:SOT23_DYY_TEX
Connections:
- net +5V: now also U3.14 (VCC)
- net GND: now also J35.S, J36.S, J37.S, J38.S, J39.S, J40.S, J41.S, J42.S, J43.S, J44.S, J45.S, J46.S, U3.7 (GND)
- new net: J39.T, U3.1 (1A)
- new net: J44.T, U3.10 (3B)
- new net: J38.T, U3.11 (4Y)
- new net: J45.T, U3.12 (4A)
- new net: J46.T, U3.13 (4B)
- new net: J40.T, U3.2 (1B)
- new net: J35.T, U3.3 (1Y)
- new net: J41.T, U3.4 (2A)
- new net: J42.T, U3.5 (2B)
- new net: J36.T, U3.6 (2Y)
- new net: J37.T, U3.8 (3Y)
- new net: J43.T, U3.9 (3A)
- no-connect marks 8 -> 42
Other:
- note added: "EHLO OPER8TRIX"

Commit message: i did a thing
Parts:
- removed J10, J11, J12, J13, J14, J15, J18, J19, J2, J20, J21, J22, J23, J24, J25, J26, J27, J28, J29, J30, J31, J32, J33, J34, J35, J36, J37, J38, J39, J40, J41, J42, J43, J44, J45, J46, J8, J9: AudioJack3_SwitchTR, AT-Footprints:CONN5_STX-3680_KYC, symbol Connector_Audio:AudioJack3_SwitchTR
- removed J16, J17: EXT MODULE, AT-Footprints:EURORACK Right Angle, symbol Connector_Generic:Conn_02x08_Odd_Even
- removed RV1, RV2: R_Potentiometer, Potentiometer_THT:Potentiometer_Bourns_PTV09A-1_Single_Vertical, symbol Device:R_Potentiometer
- removed SW3, SW4: SW_SPDT, symbol Switch:SW_SPDT
- removed U3: SN74HC32PWR, Package_SO:TSSOP-14_4.4x5mm_P0.65mm, symbol AT-Symbols:SN74HC32PWR
- added C10, C11, C12, C13, C14, C15, C16, C17, C18, C19, C26, C27: 100nF, Capacitor_SMD:C_0805_2012Metric_Pad1.18x1.45mm_HandSolder, symbol Device:C
- added C20, C23, C25, C6, C7, C9: 1uF, Capacitor_SMD:C_0805_2012Metric_Pad1.18x1.45mm_HandSolder, symbol Device:C
- added C21, C22, C24, C8: 2n2, Capacitor_SMD:C_0805_2012Metric_Pad1.18x1.45mm_HandSolder, symbol Device:C
- added D5, D6: 1N4148W, Diode_SMD:D_SOD-123, symbol Diode:1N4148W
- added J87, J88, J89, J90: AudioJack3_SwitchTR, AT-Footprints:CONN5_STX-3680_KYC, symbol Connector_Audio:AudioJack3_SwitchTR
- added Q1, Q11, Q12, Q13, Q16, Q17, Q18, Q4, Q6, Q8: BC548, Package_TO_SOT_THT:TO-92_Inline, symbol Transistor_BJT:BC548
- added Q14, Q15, Q2, Q3, Q5, Q7: BC558, Package_TO_SOT_THT:TO-92_Inline, symbol Transistor_BJT:BC558
- added R100, R101, R102, R103, R104, R105, R106, R107, R108, R109, R110, R111, R112, R113, R114, R115, R116, R117, R118, R119, R120, R121, R122, R123, R124, R125, R126, R127, R128, R129, R130, R131, R132, R133, R134, R135, R136, R21, R31, R32, R33, R34, R40, R41, R43, R44, R45, R82, R83, R84, R85, R86, R87, R88, R89, R90, R91, R92, R93, R94, R95, R96, R97, R98, R99: 20k, Resistor_SMD:R_0805_2012Metric_Pad1.20x1.40mm_HandSolder, symbol Device:R
- added R137, R139, R140, R142, R144, R146, R148, R151, R153, R159, R160, R161, R49, R55, R59, R60, R61, R64, R67, R71, R72, R75, R76, R78, R79, R81: 100k, Resistor_SMD:R_0805_2012Metric_Pad1.20x1.40mm_HandSolder, symbol Device:R
- added R138, R51, R54, R77: 33k, Resistor_SMD:R_0805_2012Metric_Pad1.20x1.40mm_HandSolder, symbol Device:R
- added R141, R74: 1k5, Resistor_SMD:R_0805_2012Metric_Pad1.20x1.40mm_HandSolder, symbol Device:R
- added R143, R145, R73, R80: 1M, Resistor_SMD:R_0805_2012Metric_Pad1.20x1.40mm_HandSolder, symbol Device:R
- added R147, R152, R68, R70: 68k, Resistor_SMD:R_0805_2012Metric_Pad1.20x1.40mm_HandSolder, symbol Device:R
- added R149, R69: 14k, Resistor_SMD:R_0805_2012Metric_Pad1.20x1.40mm_HandSolder, symbol Device:R
- added R150, R63: 47k, Resistor_SMD:R_0805_2012Metric_Pad1.20x1.40mm_HandSolder, symbol Device:R
- added R154, R155, R158, R162, R163, R19, R37, R39, R48, R50, R52, R53, R58, R62, R65, R66: 1k, Resistor_SMD:R_0805_2012Metric_Pad1.20x1.40mm_HandSolder, symbol Device:R
- added R156, R157, R20, R35, R42, R46, R56, R57: 10k, Resistor_SMD:R_0805_2012Metric_Pad1.20x1.40mm_HandSolder, symbol Device:R
- added R18, R38: 51k, Resistor_SMD:R_0805_2012Metric_Pad1.20x1.40mm_HandSolder, symbol Device:R
- added R36, R47: 200k, Resistor_SMD:R_0805_2012Metric_Pad1.20x1.40mm_HandSolder, symbol Device:R
- added RV10, RV23, RV7, RV8: 10k, Potentiometer_THT:Potentiometer_Bourns_PTV09A-1_Single_Vertical, symbol Device:R_Potentiometer
- added RV11, RV22: 250k, Potentiometer_THT:Potentiometer_Bourns_PTV09A-1_Single_Vertical, symbol Device:R_Potentiometer
- added RV12, RV19: 100k, Potentiometer_THT:Potentiometer_Runtron_RM-065_Vertical, symbol Device:R_Potentiometer_Trim
- added RV13, RV14, RV15, RV16, RV17, RV18, RV20, RV21: 100k, Potentiometer_THT:Potentiometer_Bourns_PTV09A-1_Single_Vertical, symbol Device:R_Potentiometer
- added TH1, TH2, TH3, TH4, TH5, TH6, TH7, TH8: 10k, symbol Device:Thermistor_NTC
- added TP1, TP8: C, TestPoint:TestPoint_Pad_1.0x1.0mm, symbol Connector:TestPoint
- added TP2, TP7: D, TestPoint:TestPoint_Pad_1.0x1.0mm, symbol Connector:TestPoint
- added TP3, TP6: B, TestPoint:TestPoint_Pad_1.0x1.0mm, symbol Connector:TestPoint
- added TP4, TP5: A, TestPoint:TestPoint_Pad_1.0x1.0mm, symbol Connector:TestPoint
- added U10, U13: TL074, AT-Footprints:SOT23_DYY_TEX, symbol Amplifier_Operational:TL074
- added U11: 40106, symbol 4xxx:40106
- added U12: TL074, symbol Amplifier_Operational:TL074
- added U6, U7, U8, U9: TL072, Package_SO:TSSOP-8_4.4x3mm_P0.65mm, symbol Amplifier_Operational:TL072
Connections:
- net +12V: now also C10.2, C12.2, C14.2, C16.2, C18.2, C26.2, Q11.1 (C), Q17.1 (C), R137.1, R145.1, R21.1, R33.1, R40.1, R44.1, R73.1, R76.1, RV10.3, RV13.3, RV21.3, RV23.3, U10.4 (V+), U13.4 (V+), U6.8 (V+), U7.8 (V+), U8.8 (V+), U9.8 (V+)
- net +5V: now also R82.1
- net -12V: now also C11.1, C13.1, C15.1, C17.1, C19.1, C27.1, Q14.1 (C), Q15.1 (C), R138.2, R139.2, R157.2, R31.2, R34.2, R41.2, R45.2, R57.2, R77.2, R78.2, RV13.1, RV21.1, U10.11 (V-), U13.11 (V-), U6.4 (V-), U7.4 (V-), U8.4 (V-), U9.4 (V-)
- net GND: now also C10.1, C11.2, C12.1, C13.2, C14.1, C15.2, C16.1, C17.2, C18.1, C19.2, C21.1, C22.1, C24.1, C26.1, C27.2, C8.1, Q13.3 (E), Q16.3 (E), R136.2, R148.2, R149.2, R150.2, R152.2, R159.2, R160.2, R19.2, R39.2, R49.2, R55.2, R59.2, R60.2, R63.2, R68.2, R69.2, R71.2, RV12.2, RV12.3, RV15.3, RV18.3, RV19.2, RV19.3, U12.10 (+), U12.3 (+), U7.3 (+), U7.5 (+), U8.3 (+), U8.5 (+)
- new net: R56.1, RV10.1, RV10.2
- new net: R97.2, R98.1
- new net: R98.2, R99.1
- new net: Q2.3 (E), R21.2
- new net: R74.2, RV12.1
- new net: R104.2, R105.1
- new net: R38.1, RV8.3, U6.5 (+)
- new net: J89.T, R38.2
- new net: R76.2, RV14.3
- new net: Q11.3 (E), Q12.2 (B)
- new net: R91.2, R92.1
- new net: Q12.1 (C), R56.2, R58.1
- new net: Q12.3 (E), R57.1
- new net: R140.1, TH5.1
- new net: RV20.3, TH5.2
- new net: C24.2, C25.1, R158.2
- new net: Q5.2 (B), Q6.2 (B), U6.6 (-), U6.7
- new net: R105.2, R106.1
- new net: R106.2, R107.1
- new net: C9.2, R59.1, U9.5 (+)
- new net: R77.1, RV14.1
- new net: R118.2, R119.1
- new net: R119.2, R120.1
- new net: R153.1, R154.2, U13.8
- new net: R150.1, R153.2, U13.9 (-)
- new net: Q5.1 (C), Q6.1 (C), R42.2
- new net: Q5.3 (E), R40.2
- new net: R144.1, TH8.1
- new net: C21.2, D5.1 (K), Q13.1 (C), TP3.1, U10.3 (+), U11.1
- new net: Q7.3 (E), R44.2
- new net: R69.1, R70.2, R72.1, TP2.1, U10.6 (-)
- new net: R72.2, RV13.2
- new net: R141.2, RV19.1
- new net: J88.T, R37.1
- new net: R36.2, R37.2, U8.1
- new net: R19.1, RV7.1, RV7.2
- new net: R18.1, RV7.3, U6.3 (+)
- new net: C6.1, R49.1, U12.5 (+)
- new net: R50.2, U12.6 (-), U12.7
- new net: R117.2, R118.1
- new net: R130.2, R131.1
- new net: R131.2, R132.1
- new net: R138.1, RV16.1
- new net: D5.2 (A), U11.2
- new net: R146.1, R147.2, R149.1, TP7.1, U13.6 (-)
- new net: R146.2, RV21.2
- new net: J87.T, R18.2
- new net: R128.2, R129.1
- new net: R129.2, R130.1
- new net: C7.1, R55.1, U12.12 (+)
- new net: C7.2, R54.2, U12.8
- new net: R163.2, U12.13 (-), U12.14
- new net: R85.2, R86.1
- new net: R86.2, R87.1
- new net: Q1.3 (E), R31.1
- new net: R151.1, R152.1, U13.12 (+)
- new net: R155.2, U13.13 (-), U13.14
- new net: R142.1, TH6.1
- new net: R142.2, RV16.2
- new net: R100.1, R99.2
- new net: R100.2, R101.1
- new net: R82.2, R83.1
- new net: R83.2, R84.1
- new net: Q4.3 (E), R34.1
- new net: R20.1, R32.1, U7.2 (-)
- new net: Q1.1 (C), Q2.1 (C), R20.2
- new net: Q18.3 (E), R157.1
- new net: C22.2, D6.1 (K), Q16.1 (C), TP6.1, U11.3, U13.3 (+)
- new net: D6.2 (A), U11.4
- new net: R134.2, R135.1
- new net: R135.2, R136.1
- new net: R124.2, R125.1
- new net: Q15.3 (E), Q16.2 (B), R145.2, TP5.1
- new net: Q1.2 (B), Q2.2 (B), U6.1, U6.2 (-)
- new net: R101.2, R102.1
- new net: J90.T, R48.1
- new net: Q18.1 (C), R156.2, R158.1
- new net: R75.1, TH4.1
- new net: Q14.2 (B), R74.1, RV17.1, RV17.2, TH2.2, TH3.2, TH4.2
- new net: C20.2, U10.1, U10.2 (-)
- new net: R53.1, R54.1, U12.9 (-)
- new net: R111.2, R112.1
- new net: R112.2, R113.1
- new net: R108.2, R109.1
- new net: R109.2, R110.1
- new net: Q15.2 (B), R141.1, RV20.1, RV20.2, TH6.2, TH7.2, TH8.2
- new net: R46.1, R47.1, U8.6 (-)
- new net: R47.2, R48.2, U8.7
- new net: R127.2, R128.1
- new net: R81.1, TH1.1
- new net: R60.1, R61.2, U9.6 (-)
- new net: R78.1, RV15.1
- new net: R80.2, RV15.2
- new net: C25.2, R159.1, U9.3 (+)
- new net: Q13.2 (B), Q14.3 (E), R73.2, TP4.1
- new net: Q17.3 (E), Q18.2 (B)
- new net: R113.2, R114.1
- new net: R156.1, RV23.1, RV23.2
- new net: R87.2, R88.1
- new net: R88.2, R89.1
- new net: R70.1, RV11.1, RV11.2
- new net: R65.2, U10.13 (-), U10.14
- new net: R102.2, R103.1
- new net: C23.1, R148.1, TP8.1, U13.10 (+), U13.5 (+)
- new net: R121.2, R122.1
- new net: R122.2, R123.1
- new net: R126.2, R127.1
- new net: R61.1, R62.2, U9.7
- new net: R110.2, R111.1
- new net: R95.2, R96.1
- new net: R96.2, R97.1
- new net: Q7.1 (C), Q8.1 (C), R46.2
- new net: Q7.2 (B), Q8.2 (B), R43.2, U7.7
- new net: R35.1, R36.1, U8.2 (-)
- new net: C6.2, R51.2, U12.1
- new net: C20.1, R71.1, TP1.1, U10.10 (+), U10.5 (+)
- new net: R64.1, R66.2, U10.8
- new net: R63.1, R64.2, U10.9 (-)
- new net: R123.2, R124.1
- new net: R42.1, R43.1, U7.6 (-)
- new net: R107.2, R108.1
- new net: R147.1, RV22.1, RV22.2
- new net: C23.2, U13.1, U13.2 (-)
- new net: R132.2, R133.1
- new net: R133.2, R134.1
- new net: R80.1, TH3.1
- new net: R89.2, R90.1
- new net: R90.2, R91.1
- new net: R75.2, RV14.2
- new net: Q8.3 (E), R45.1
- new net: R139.1, RV18.1
- new net: R143.2, RV18.2
- new net: R93.2, R94.1
- new net: R67.1, R68.1, U10.12 (+)
- new net: R84.2, R85.1
- new net: R143.1, TH7.1
- new net: R79.1, TH2.1
- new net: R67.2, U10.7
- new net: R161.1, R162.2, U9.1
- new net: R116.2, R117.1
- new net: C8.2, C9.1, R58.2
- new net: R160.1, R161.2, U9.2 (-)
- new net: Q3.1 (C), Q4.1 (C), R35.2
- new net: Q3.2 (B), Q4.2 (B), R32.2, U7.1
- new net: Q3.3 (E), R33.2
- new net: RV17.3, TH1.2
- new net: R120.2, R121.1
- new net: R137.2, RV16.3
- new net: R51.1, R52.1, U12.2 (-)
- new net: R94.2, R95.1
- new net: Q6.3 (E), R41.1
- new net: R151.2, U13.7
- new net: R39.1, RV8.1, RV8.2
- new net: R115.2, R116.1
- new net CV1: R144.2, R79.2
- new net FM1: R140.2, R81.2
- new net Note C1: R125.2, R126.1
- new net Note C2: R114.2, R115.1
- new net Note C3: R103.2, R104.1
- new net Note C4: R92.2, R93.1
- new net PWM IN 1: RV11.3
- new net PWM IN 2: RV22.3
- new net PWM1: R65.1
- new net PWM2: R155.1
- new net SAW1: Q11.2 (B), R66.1
- new net SAW2: Q17.2 (B), R154.1
- new net TRI1: J87.TN, R62.1
- new net TRI2: J89.TN, R162.1
- new net VCF1 OUT: R50.1
- new net VCF2 OUT: R163.1
- no-connect marks 42 -> 6
Other:
- added sheet Octuple Or (octor.kicad_sch)
- added sheet Scope (scope.kicad_sch)
- added sheet USB (usb.kicad_sch)
- added sheet dialpad (dialpad.kicad_sch)
- note added: "CV 1v/Octave REF"
- note added: "I stole this from Moritz Klein over at Erica synths https://www.ericasynths.lv/shop/diy-kits-1/edu-diy-vco/ https://www.ericasynths.lv/shop/diy-kits-1/edu-diy-wavefolder/"
- note added: "I stole this from Moritz Klein over at Erica syntsh https://www.ericasynths.lv/shop/diy-kits-1/edu-diy-vco/"
- note added: "Twin Triple VCO w/ Wavefolders"
- note removed: "EHLO OPER8TRIX"
- moved on the sheet: J5, J6, J7, R13, R14, R15, R16, R17, R22, R23, R24, R25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
