File: Essential/Essential.kicad_pcb (KiCad board)
At the start: 2 copper layers, 99.5 x 101.5 mm, 54 parts, among them J1 Bus_EURO_Express, J1 EURO_EXPRESS, J2 10025026-10103TLF, J3 EURO_CONN, J5 ATX_POWER, J6 FRONT_PANEL, SW1 CH559_PRG, U1 DKA30A-12, U2 MAX16054, U4 TMUX4051PWR, U5 U_RP2040, U6 W25Q32JVSS, X1 12MHz

Commit message: i did a thing
Parts:
- removed C1: 0.1uF, Capacitor_SMD:C_0805_2012Metric_Pad1.18x1.45mm_HandSolder
- removed C10, C11, C12, C13, C14, C15, C7, C8, C9: 0.1uF, llama_shared:C_0402_1005Metric
- removed C16, C17: 1uF, llama_shared:C_0402_1005Metric
- removed C18, C19: 30pF, llama_shared:C_0402_1005Metric
- removed C2: 10uF, Capacitor_SMD:C_0805_2012Metric_Pad1.18x1.45mm_HandSolder
- removed C3, C4, C5, C6: 100uF, llama_shared:C_1210_3225Metric
- removed H1, H5 (x2), H6 (x2), H7 (x2), H8: H_HOLE, llama_shared:H_ATX_PERF
- removed J1: EURO_EXPRESS, AT-Footprints:BUS_EUROexpress
- removed J1: Bus_EURO_Express, Connector_PCBEdge:BUS_PCIexpress_x16
- removed J2 (x2): 10025026-10103TLF, AT-Footprints:AMPHENOL_10025026-10103TLF
- removed J3: EURO_CONN, AT-Footprints:EURORACK Right Angle
- removed J5: ATX_POWER, ATX:ATX_24_RIGHT_ANGLE_MOLEX_469911024
- removed J6: FRONT_PANEL, llama_shared:P_CONN_PANEL
- removed R1: 10k, Resistor_SMD:R_0805_2012Metric_Pad1.20x1.40mm_HandSolder
- removed R10, R12: 1k, llama_shared:R_0402_1005Metric
- removed R11, R9: 10k, llama_shared:R_0402_1005Metric
- removed R2, R4, R5, R6, R7: 470, Resistor_SMD:R_0805_2012Metric_Pad1.20x1.40mm_HandSolder
- removed R3, R8: 330, Resistor_SMD:R_0805_2012Metric_Pad1.20x1.40mm_HandSolder
- removed SW1: CH559_PRG, llama_shared:SW_B3FS-1010
- removed U1: DKA30A-12, AT-Footprints:DKA30_MWU
- removed U2: MAX16054, llama_shared:U_TSOT-23-6
- removed U4: TMUX4051PWR, AT-Footprints:TSSOP16_PW_TEX
- removed U5: U_RP2040, llama_shared:U_QFN40P700X700X90-57N
- removed U6: W25Q32JVSS, llama_shared:U_SOIC-8_5.23x5.23mm_P1.27mm
- removed X1: 12MHz, llama_shared:X_SMD3225
- added C21: 1uF, Capacitor_SMD:C_0805_2012Metric_Pad1.18x1.45mm_HandSolder, F.Cu at (110.7, 52.7)
- added C22: 5.6nF, Capacitor_SMD:C_0805_2012Metric_Pad1.18x1.45mm_HandSolder, F.Cu at (110.7, 55.8)
- added C23: 2.2nF, Capacitor_SMD:C_0805_2012Metric_Pad1.18x1.45mm_HandSolder, F.Cu at (110.7, 58.8)
- added C24: 680p, Capacitor_SMD:C_0805_2012Metric_Pad1.18x1.45mm_HandSolder, F.Cu at (110.7, 61.8)
- added C25: 680pF, Capacitor_SMD:C_0805_2012Metric_Pad1.18x1.45mm_HandSolder, F.Cu at (110.7, 64.8)
- added C26: 2.2nF, Capacitor_SMD:C_0805_2012Metric_Pad1.18x1.45mm_HandSolder, F.Cu at (110.7, 67.8)
- added C27: 5.6nF, Capacitor_SMD:C_0805_2012Metric_Pad1.18x1.45mm_HandSolder, F.Cu at (110.7, 70.8)
- added Q7: BC548, Package_TO_SOT_SMD:SOT-23, F.Cu at (137.7, 81.7)
- added Q8: BC548, Package_TO_SOT_SMD:SOT-23, F.Cu at (115.1, 75.0)
- added R100: 20k, Resistor_SMD:R_0805_2012Metric_Pad1.20x1.40mm_HandSolder, F.Cu at (125.0, 61.5)
- added R101: 470k, Resistor_SMD:R_0805_2012Metric_Pad1.20x1.40mm_HandSolder, F.Cu at (125.0, 64.5)
- added R102: 100k, Resistor_SMD:R_0805_2012Metric_Pad1.20x1.40mm_HandSolder, F.Cu at (129.8, 49.7)
- added R103: 22k, Resistor_SMD:R_0805_2012Metric_Pad1.20x1.40mm_HandSolder, F.Cu at (129.8, 52.6)
- added R104: 33k, Resistor_SMD:R_0805_2012Metric_Pad1.20x1.40mm_HandSolder, F.Cu at (129.8, 55.6)
- added R105: 100k, Resistor_SMD:R_0805_2012Metric_Pad1.20x1.40mm_HandSolder, F.Cu at (129.8, 58.5)
- added R106: 1k, Resistor_SMD:R_0805_2012Metric_Pad1.20x1.40mm_HandSolder, F.Cu at (129.8, 61.5)
- added R107: 1k, Resistor_SMD:R_0805_2012Metric_Pad1.20x1.40mm_HandSolder, F.Cu at (129.8, 64.5)
- added R84: 100k, Resistor_SMD:R_0805_2012Metric_Pad1.20x1.40mm_HandSolder, F.Cu at (115.5, 49.7)
- added R85: 100k, Resistor_SMD:R_0805_2012Metric_Pad1.20x1.40mm_HandSolder, F.Cu at (115.5, 52.6)
- added R86: 100k, Resistor_SMD:R_0805_2012Metric_Pad1.20x1.40mm_HandSolder, F.Cu at (115.5, 55.6)
- added R87: 100k, Resistor_SMD:R_0805_2012Metric_Pad1.20x1.40mm_HandSolder, F.Cu at (115.5, 58.5)
- added R88: 680R, Resistor_SMD:R_0805_2012Metric_Pad1.20x1.40mm_HandSolder, F.Cu at (115.5, 61.5)
- added R89: 680R, Resistor_SMD:R_0805_2012Metric_Pad1.20x1.40mm_HandSolder, F.Cu at (115.5, 64.5)
- added R90: 100k, Resistor_SMD:R_0805_2012Metric_Pad1.20x1.40mm_HandSolder, F.Cu at (120.3, 49.7)
- added R91: 100k, Resistor_SMD:R_0805_2012Metric_Pad1.20x1.40mm_HandSolder, F.Cu at (120.3, 52.6)
- added R92: 1k, Resistor_SMD:R_0805_2012Metric_Pad1.20x1.40mm_HandSolder, F.Cu at (120.3, 55.6)
- added R93: 1k, Resistor_SMD:R_0805_2012Metric_Pad1.20x1.40mm_HandSolder, F.Cu at (120.3, 58.5)
- added R94: 100k, Resistor_SMD:R_0805_2012Metric_Pad1.20x1.40mm_HandSolder, F.Cu at (120.3, 61.5)
- added R95: 4k7, Resistor_SMD:R_0805_2012Metric_Pad1.20x1.40mm_HandSolder, F.Cu at (120.3, 64.5)
- added R96: 1M, Resistor_SMD:R_0805_2012Metric_Pad1.20x1.40mm_HandSolder, F.Cu at (125.0, 49.7)
- added R97: 470k, Resistor_SMD:R_0805_2012Metric_Pad1.20x1.40mm_HandSolder, F.Cu at (125.0, 52.6)
- added R98: 10k, Resistor_SMD:R_0805_2012Metric_Pad1.20x1.40mm_HandSolder, F.Cu at (125.0, 55.6)
- added R99: 47k, Resistor_SMD:R_0805_2012Metric_Pad1.20x1.40mm_HandSolder, F.Cu at (125.0, 58.5)
- added U9: TL074, Package_SO:TSSOP-14_4.4x5mm_P0.65mm, F.Cu at (150.0, 77.2)
- C20: value 0.1uF -> 1uF; footprint llama_shared:C_0402_1005Metric -> Capacitor_SMD:C_0805_2012Metric_Pad1.18x1.45mm_HandSolder
- moved C20 179.0 mm to (110.7, 49.7)
Connections:
- C20 pad 1: GND -> Net-(Q7-E)
- C20 pad 2: RP_3.3V -> Net-(U9A-+)
Routing:
- net +12V: track 103.9 -> 0.00 mm
- net +3.3V: track 69.5 -> 0.00 mm
- net VCC: track 68.8 -> 0.00 mm
- net +5VSB: track 61.1 -> 0.00 mm, vias 1 -> 0
- net /~{PS_ON}: track 28.8 -> 0.00 mm
- net -12V: track 16.1 -> 0.00 mm
- net /~{RST_SW}: track 10.9 -> 0.00 mm
- net /~{PWR_SW}: track 9.16 -> 0.00 mm
- net /PWR_LED-: track 7.73 -> 0.00 mm
- net /HDD_LED+: track 5.04 -> 0.00 mm
- net GND: track 3.92 -> 0.00 mm
- net /HDD_LED-: track 3.90 -> 0.00 mm
- net /~{RST_SIG}: track 3.89 -> 0.00 mm
- net /PWR_LED+: track 3.76 -> 0.00 mm
- net /GATE: track 2.54 -> 0.00 mm
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- removed copper zone on B.Cu, net GND
Other:
- board outline removed
