File: Essential/Essential.kicad_sch (KiCad schematic)
At the start: 19 parts, among them J1 EURO_CONN, J10 AUDIO 1 OUT, J11 AUDIO 2 OUT, J12 AUDIO 1 IN, J13 AUDIO 2 IN, J2 EXT MODULE #1, J3 NOISE OUT, J4 EXT MODULE #1, J5 CV OUT, J6 GATE IN, J7 GATE OUT, J8 CV IN, J9 TRIG IN

Commit message: i did a thing
Parts:
- removed D1: 5V OK, LED_SMD:LED_0805_2012Metric, symbol Device:LED
- removed D2: 12V OK, LED_SMD:LED_0805_2012Metric, symbol Device:LED
- removed D3: -12V OK, LED_SMD:LED_0805_2012Metric, symbol Device:LED
- removed J1: EURO_CONN, AT-Footprints:EURORACK Right Angle, symbol Connector_Generic:Conn_02x08_Odd_Even
- removed J10: AUDIO 1 OUT, Connector_Audio:Jack_3.5mm_Ledino_KB3SPRS_Horizontal, symbol Connector_Audio:AudioJack3
- removed J11: AUDIO 2 OUT, Connector_Audio:Jack_3.5mm_Ledino_KB3SPRS_Horizontal, symbol Connector_Audio:AudioJack3
- removed J12: AUDIO 1 IN, Connector_Audio:Jack_3.5mm_Ledino_KB3SPRS_Horizontal, symbol Connector_Audio:AudioJack3
- removed J13: AUDIO 2 IN, Connector_Audio:Jack_3.5mm_Ledino_KB3SPRS_Horizontal, symbol Connector_Audio:AudioJack3
- removed J2, J4: EXT MODULE #1, AT-Footprints:EURORACK Right Angle, symbol Connector_Generic:Conn_02x08_Odd_Even
- removed J3: NOISE OUT, Connector_Audio:Jack_3.5mm_Ledino_KB3SPRS_Horizontal, symbol Connector_Audio:AudioJack3
- removed J5: CV OUT, Connector_Audio:Jack_3.5mm_Ledino_KB3SPRS_Horizontal, symbol Connector_Audio:AudioJack3
- removed J6: GATE IN, Connector_Audio:Jack_3.5mm_Ledino_KB3SPRS_Horizontal, symbol Connector_Audio:AudioJack3
- removed J7: GATE OUT, Connector_Audio:Jack_3.5mm_Ledino_KB3SPRS_Horizontal, symbol Connector_Audio:AudioJack3
- removed J8: CV IN, Connector_Audio:Jack_3.5mm_Ledino_KB3SPRS_Horizontal, symbol Connector_Audio:AudioJack3
- removed J9: TRIG IN, Connector_Audio:Jack_3.5mm_Ledino_KB3SPRS_Horizontal, symbol Connector_Audio:AudioJack3
- removed R2: 500, Resistor_SMD:R_0805_2012Metric_Pad1.20x1.40mm_HandSolder, symbol Device:R
- added C1, C2, C3, C4, C5, C6: 100nF, Capacitor_SMD:C_0805_2012Metric_Pad1.18x1.45mm_HandSolder, symbol Device:C
- added D4: PRSNT, LED_SMD:LED_0805_2012Metric, symbol Device:LED
- added D5: 5V OK, LED_SMD:LED_0805_2012Metric, symbol Device:LED
- added D6: 12V OK, LED_SMD:LED_0805_2012Metric, symbol Device:LED
- added D7: -12V OK, LED_SMD:LED_0805_2012Metric, symbol Device:LED
- added J1: Folder, Connector_Audio:Jack_3.5mm_CUI_SJ-3524-SMT_Horizontal, symbol Connector_Audio:AudioJack2_SwitchT
- added J14: OPT EURO, AT-Footprints:EURORACK Right Angle, symbol Connector_Generic:Conn_02x08_Odd_Even
- added J15: DIN41612_02x32_AB, symbol Connector:DIN41612_02x32_AB
- added J2: Fold, Connector_Audio:Jack_3.5mm_CUI_SJ-3524-SMT_Horizontal, symbol Connector_Audio:AudioJack2_SwitchT
- added J20: ~, Connector_PCBEdge:BUS_PCIexpress_x4, symbol AT-Symbols:EURO_Express_x4
- added J3, J4: Laundry, Connector_Audio:Jack_3.5mm_CUI_SJ-3524-SMT_Horizontal, symbol Connector_Audio:AudioJack2_SwitchT
- added J5: Triangle, Connector_Audio:Jack_3.5mm_CUI_SJ-3524-SMT_Horizontal, symbol Connector_Audio:AudioJack2_SwitchT
- added J6: Saw, Connector_Audio:Jack_3.5mm_CUI_SJ-3524-SMT_Horizontal, symbol Connector_Audio:AudioJack2_SwitchT
- added J7: PWM, Connector_Audio:Jack_3.5mm_CUI_SJ-3524-SMT_Horizontal, symbol Connector_Audio:AudioJack2_SwitchT
- added J8: Triange Gen, Connector_Audio:Jack_3.5mm_CUI_SJ-3524-SMT_Horizontal, symbol Connector_Audio:AudioJack2_SwitchT
- added R4, R5: 150, Resistor_SMD:R_0805_2012Metric_Pad1.20x1.40mm_HandSolder, symbol Device:R
- added R6, R7: 500, Resistor_SMD:R_0805_2012Metric_Pad1.20x1.40mm_HandSolder, symbol Device:R
- added R8: 1k, Resistor_SMD:R_0805_2012Metric_Pad1.20x1.40mm_HandSolder, symbol Device:R
- added RV1, RV2: 10k, Potentiometer_THT:Potentiometer_Bourns_PTV09A-2_Single_Horizontal, symbol Device:R_Potentiometer
- added U11, U12, U13: TL072, Package_SO:TSSOP-8_4.4x3mm_P0.65mm, symbol Amplifier_Operational:TL072
- R1: value 150 -> 1k
- R3: value 500 -> 1k
Connections:
- net +12v: now also C1.2, C3.2, C5.2, J14.10 (Pin_10), J14.9 (Pin_9), J15.a4 (Pin_a4), J15.b4 (Pin_b4), U11.8 (V+), U12.8 (V+), U13.8 (V+)
- net +5: now also J14.11 (Pin_11), J14.12 (Pin_12), J15.a2 (Pin_a2), J15.b2 (Pin_b2)
- net -12v: now also C2.1, C4.1, C6.1, J14.1 (Pin_1), J14.2 (Pin_2), J15.a7 (Pin_a7), J15.b7 (Pin_b7), U11.4 (V-), U12.4 (V-), U13.4 (V-)
- net CON_CV 0: now also J15.a10 (Pin_a10)
- net CON_GATE 0: now also J15.a9 (Pin_a9)
- net GND: now also C1.1, C2.2, C3.1, C4.2, C5.1, C6.2, J1.S, J14.3 (Pin_3), J14.4 (Pin_4), J14.5 (Pin_5), J14.6 (Pin_6), J14.7 (Pin_7), J14.8 (Pin_8), J15.a11 (Pin_a11), J15.a15 (Pin_a15), J15.a17 (Pin_a17), J15.a19 (Pin_a19), J15.a21 (Pin_a21), J15.a23 (Pin_a23), J15.a26 (Pin_a26), J15.a3 (Pin_a3), J15.a5 (Pin_a5), J15.a6 (Pin_a6), J15.a8 (Pin_a8), J15.b1 (Pin_b1), J15.b11 (Pin_b11), J15.b13 (Pin_b13), J15.b14 (Pin_b14), J15.b16 (Pin_b16), J15.b18 (Pin_b18), J15.b20 (Pin_b20), J15.b26 (Pin_b26), J15.b3 (Pin_b3), J15.b32 (Pin_b32), J15.b5 (Pin_b5), J15.b6 (Pin_b6), J15.b8 (Pin_b8), J2.S, J20.A3 (GND), J20.A5 (GND), J20.A6 (GND), J20.A8 (GND), J20.B1 (GND), J20.B3 (GND), J20.B5 (GND), J20.B6 (GND), J20.B8 (GND), J3.S, J4.S, J5.S, J6.S, J7.S, J8.S, R5.1, R6.1, R7.2, R8.2
- net at R1.1: now also J4.T
- net FOLD_2_OUT: now reaches R1.2
- net at R3.1: now also RV1.1, RV1.2
- new net: D5.1 (K), R5.2
- new net: D4.1 (K), R4.2
- new net: D4.2 (A), J20.B31 (PRSNT_B)
- new net: R8.1, RV2.1, RV2.2
- new net: J20.A1 (PRSNT_A), R4.1
- new net: D6.1 (K), R6.2
- new net: D7.2 (A), R7.1
- new net +12V: D6.2 (A), J20.A4 (+12V), J20.B4 (+12V)
- new net +5V: D5.2 (A), J20.A2 (+5V), J20.B2 (+5V)
- new net -12V: D7.1 (K), J20.A7 (-12V), J20.B7 (-12V)
- new net 5V Port 1: J15.a12 (Pin_a12)
- new net Audio_IN_A: J15.b15 (Pin_b15)
- new net Audio_IN_B: J15.b17 (Pin_b17)
- new net Audio_IN_C: J15.b19 (Pin_b19)
- new net Audio_IN_D: J15.b21 (Pin_b21)
- new net Audio_OUT_A: J15.a14 (Pin_a14)
- new net Audio_OUT_B: J15.a16 (Pin_a16)
- new net Audio_OUT_C: J15.a18 (Pin_a18)
- new net Audio_OUT_D: J15.a20 (Pin_a20)
- new net BUSY: J15.a31 (Pin_a31)
- new net CON_CV: J14.13 (Pin_13), J14.14 (Pin_14)
- new net CON_GATE: J14.15 (Pin_15), J14.16 (Pin_16)
- new net D+ Port 1: J15.b12 (Pin_b12)
- new net D- Port 1: J15.a13 (Pin_a13)
- new net FOLD_1_CTRL_1: RV1.3
- new net FOLD_1_IN: J1.T
- new net FOLD_1_OUT: J3.T
- new net FOLD_2_CTRL_1: RV2.3
- new net FOLD_2_IN: J2.T
- new net GPIO 1: J15.a28 (Pin_a28)
- new net GPIO 2: J15.a29 (Pin_a29)
- new net GPIO 3: J15.a30 (Pin_a30)
- new net GPIO 4: J15.b28 (Pin_b28)
- new net GPIO 5: J15.b29 (Pin_b29)
- new net GPIO 6: J15.b30 (Pin_b30)
- new net I2C ID0: J15.b24 (Pin_b24)
- new net I2C ID1: J15.a25 (Pin_a25)
- new net I2C ID2: J15.b25 (Pin_b25)
- new net I2C SCL: J15.b23 (Pin_b23)
- new net I2C SDA: J15.a24 (Pin_a24)
- new net I2C2 SCL: J15.a27 (Pin_a27)
- new net I2C2 SDA: J15.b27 (Pin_b27)
- new net OUT_CV 0: J15.b10 (Pin_b10)
- new net OUT_GATE 0: J15.b9 (Pin_b9)
- new net PRSNT_A: J15.a1 (Pin_a1)
- new net PRSNT_B: J15.b31 (Pin_b31)
- new net PWM1: J7.T
- new net READY: J15.a32 (Pin_a32)
- new net S2T_IN_1: J8.T
- new net SAW1: J6.T
- new net SAW_1: J8.TN
- new net TRI_1: J1.TN, J5.T
- new net TRI_2: J2.TN
- new net UART RX: J15.b22 (Pin_b22)
- new net UART TX: J15.a22 (Pin_a22)
- no-connect marks 6 -> 5
Other:
- added sheet Filter Stage (Filter.kicad_sch)
- added sheet Oscillators (Oscillators.kicad_sch)
- added sheet Output Stage (Output.kicad_sch)
- added sheet Utility (Utility.kicad_sch)
- note added: "Audio I/O Bus"
- note added: "Euro Power"
- note added: "GPIO and Status"
- note added: "I2C and UART"
- note added: "Notch"
- note added: "USB"
- note removed: "Pull shrouded RA conn for this"
- company: (none) -> velvia-fifty
- title: (none) -> Laundromat
