File: PSU/PSU.kicad_sch (KiCad schematic)
At the start: 40 parts, among them J1 EXT USB C, J10 EURO_CONN, J11 EURO_CONN, J12 EURO_CONN, J2 OPT_DC, J3 EURO_CONN, J4 INT_USB, J5 EURO_CONN, J6 EURO_CONN, J7 EURO_CONN, J8 EURO_CONN, J9 EURO_CONN, Q1 2N3904, U1 DKA30A-12, U7 STUSB4500QTR, U8 LM2596T-12, U9 LM2596T-12

Commit message: i did a thing
Parts:
- added U2: STUSB4761QTR, AT-Footprints:QFN16_STUSB4761QTR_STM, symbol AT-Symbols:STUSB4761QTR
Other:
- note added: "USB PD 20V - Sink"
- note added: "WATTER SPORTS"
- note removed: "USB PD 20V"
Changed lines of the file:
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@@
 		)
 	)
+	(text_box "8-5 on Datasheet"
+		(exclude_from_sim no)
+		(at 370.84 153.67 0)
+		(size 39.37 30.48)
+		(stroke
+			(width 0)
+			(type default)
+		)
+		(fill
+			(type none)
+		)
+		(effects
+			(font
+				(size 1.27 1.27)
+			)
+			(justify left top)
+		)
+	)
 	(text_box "ATX To -12???\n"
 		(exclude_from_sim no)
@@
 		)
 	)
-	(text "USB PD 20V"
+	(text "USB PD 20V - Sink"
 		(exclude_from_sim no)
-		(at 225.044 213.614 0)
+		(at 240.03 216.154 0)
 		(effects
 			(font
@@
 		)
 	)
+	(text "WATTER\nSPORTS"
+		(exclude_from_sim no)
+		(at 107.696 67.564 0)
+		(effects
+			(font
+				(face "Boston Traffic")
+				(size 5.08 5.08)
+			)
+		)
+	)
 	(text "Regulated Power"
 		(exclude_from_sim no)
@@
 					(unit 1)
 				)
+			)
+		)
+	)
+	(symbol
+		(lib_id "AT-Symbols:STUSB4761QTR")
+		(at 299.72 384.81 0)
+		(unit 1)
+		(exclude_from_sim no)
+		(in_bom yes)
+		(on_board yes)
+		(dnp no)
+		(fields_autoplaced yes)
+		(property "Reference" "U2"
+			(at 337.82 374.65 0)
+			(effects
+				(font
+					(size 1.524 1.524)
+				)
+			)
+		)
+		(property "Value" "STUSB4761QTR"
+			(at 337.82 377.19 0)
+			(effects
+				(font
+					(size 1.524 1.524)
+				)
+			)
+		)
+		(property "Footprint" "AT-Footprints:QFN16_STUSB4761QTR_STM"
+			(at 302.768 370.84 0)
+			(effects
+				(font
+					(size 1.27 1.27)
+					(italic yes)
+				)
+				(hide yes)
+			)
+		)
+		(property "Datasheet" "STUSB4761QTR"
+			(at 299.72 374.396 0)
+			(effects
+				(font
+					(size 1.27 1.27)
+					(italic yes)
+				)
+				(hide yes)
+			)
+		)
+		(property "Description" ""
+			(at 299.72 384.81 0)
+			(effects
+				(font
+					(size 1.27 1.27)
+				)
+				(hide yes)
+			)
+		)
+		(pin "2"
+		)
+		(pin "13"
+		)
+		(pin "11"
+		)
+		(pin "12"
+		)
+		(pin "1"
+		)
+		(pin "5"
+		)
+		(pin "16"
+		)
+		(pin "15"
+		)
+		(pin "7"
+		)
+		(pin "10"
+		)
+		(pin "8"
+		)
+		(pin "4"
+		)
+		(pin "14"
+		)
+		(pin "3"
+		)
+		(pin "9"
+		)
+		(pin "6"
+		)
+		(instances
+			(project ""
+				(path "/b48a24c3-e448-4ffe-b89b-bee99abc70c9"
+					(reference "U2")
+					(unit 1)
+				)
