File: Modules/One-8-DM5/Mechanical.kicad_sch (KiCad schematic)
At the start: 16 parts

Commit message: big old push of morphine to commit war crimes
Parts:
- removed H10, H11, H12, H13, H14, H15, H16, H7, H8, H9: Mousebite, mousebites:mouse-bite-2mm-slot, symbol Mechanical:MountingHole
- added FID1, FID2, FID3, FID4: Fiducial, Fiducial:Fiducial_1mm_Mask3mm, symbol Mechanical:Fiducial
- added H17, H18, H19, H20: Panel Hole, AT-Footprints:Panel - Hole, symbol Mechanical:MountingHole
