File: Modules/One-8-DM5/One-8-DM5.kicad_pcb (KiCad board)
At the start: 2 copper layers, 100 x 94 mm, 59 parts, among them J1 ALPHA, J10 Why B 0, J12 Why C 0, J13 Stereo 0, J15 Stereo 1, J16 Stereo 2, J17 Stereo 3, J18 Stereo 4, J19 Stereo 5, J2 ALPHA, J20 Stereo 6, J21 Stereo 7, J22 Stereo 8, J23 HDMI, J24 Mono, J25 Why A 1, J26 Why B 1, J27 Why C 1, J28 Why A 3, J29 GAMMA, J3 ALPHA, J30 Why B 3, J31 Why C 3, J32 GAMMA, J33 DELTA, J34 Why A 2, J35 Why B 2, J36 Why C 2, J37 C/D, J38 C/D, J39 C/D, J4 BETA, J5 A/B, J6 A/B, J7 A/B, J8 A/GAMMA, J9 Why A 0

Commit message: big old push of morphine to commit war crimes
Parts:
- removed H10, H11, H12, H13, H14, H15, H16, H7, H8, H9: Mousebite, mousebites:mouse-bite-2mm-slot
- added FID1: Fiducial, Fiducial:Fiducial_1mm_Mask2mm, F.Cu at (131.1, 48.7)
- added FID2: Fiducial, Fiducial:Fiducial_1mm_Mask3mm, F.Cu at (218.4, 48.7)
- added FID3: Fiducial, Fiducial:Fiducial_1mm_Mask3mm, F.Cu at (131.1, 141.0)
- added FID4: Fiducial, Fiducial:Fiducial_1mm_Mask2mm, F.Cu at (218.4, 141.0)
- added H17: Panel Hole, AT-Footprints:Panel - Hole, F.Cu at (127.3, 47.3)
- added H18: Panel Hole, AT-Footprints:Panel - Hole, F.Cu at (222.3, 47.3)
- added H19: Panel Hole, AT-Footprints:Panel - Hole, F.Cu at (127.3, 142.4)
- added H20: Panel Hole, AT-Footprints:Panel - Hole, F.Cu at (222.3, 142.4)
- added J11: EXT_INTERFACE_1, AT-Footprints:AMPHENOL_SFV30R-4STE1HLF - FFC - 30 RA, F.Cu at (105.9, 104.6)
- added J14: Daughter, AT-Footprints:AMPHENOL_SFV30R-4STE1HLF - FFC - 30 RA, F.Cu at (105.9, 113.3)
- moved G1 3.96 mm to (138.9, 72.7)
- moved G2 3.96 mm to (148.9, 74.7)
- moved H1 3.96 mm to (129.8, 74.8)
- moved H2 3.96 mm to (219.8, 74.8)
- moved J23 3.96 mm to (213.4, 56.7)
- moved J13 3.96 mm to (132.6, 55.7)
- moved J15 3.96 mm to (138.9, 55.7)
- moved J16 3.96 mm to (145.1, 55.7)
- moved J17 3.96 mm to (151.4, 55.7)
- moved J18 3.96 mm to (157.6, 55.7)
- moved J19 3.96 mm to (163.9, 55.7)
- moved J20 3.96 mm to (170.1, 55.7)
- moved J21 3.96 mm to (176.4, 55.7)
- moved J22 3.96 mm to (182.6, 55.7)
- moved J24 3.96 mm to (195.1, 55.7)
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Other:
- board size 100 x 94 mm -> 103.5 x 100 mm
- board text added: "V-CUT"
