File: Modules/Superstitious Acrobat/Superstitious Acrobat.kicad_sch (KiCad schematic)
At the start: 2 parts, among them J11 EXT_INTERFACE_1, J14 Daughter

Commit message: big old push of morphine to commit war crimes
Other:
- moved on the sheet: J14
Changed lines of the file:
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@@
 	)
 	(label "DB PIN 8"
-		(at 284.48 251.46 180)
+		(at 308.61 248.92 180)
 		(fields_autoplaced yes)
 		(effects
@@
 	)
 	(label "DB PIN 28"
-		(at 284.48 302.26 180)
+		(at 308.61 299.72 180)
 		(fields_autoplaced yes)
 		(effects
@@
 	)
 	(label "DB PIN 20"
-		(at 284.48 281.94 180)
+		(at 308.61 279.4 180)
 		(fields_autoplaced yes)
 		(effects
@@
 	)
 	(label "DB PIN 11"
-		(at 284.48 259.08 180)
+		(at 308.61 256.54 180)
 		(fields_autoplaced yes)
 		(effects
@@
 	)
 	(label "DB PIN 14"
-		(at 284.48 266.7 180)
+		(at 308.61 264.16 180)
 		(fields_autoplaced yes)
 		(effects
@@
 	)
 	(label "DB PIN 24"
-		(at 284.48 292.1 180)
+		(at 308.61 289.56 180)
 		(fields_autoplaced yes)
 		(effects
@@
 	)
 	(label "DB PIN 3"
-		(at 284.48 238.76 180)
+		(at 308.61 236.22 180)
 		(fields_autoplaced yes)
 		(effects
@@
 	)
 	(label "DB PIN 13"
-		(at 284.48 264.16 180)
+		(at 308.61 261.62 180)
 		(fields_autoplaced yes)
 		(effects
@@
 	)
 	(label "DB PIN 18"
-		(at 284.48 276.86 180)
+		(at 308.61 274.32 180)
 		(fields_autoplaced yes)
 		(effects
@@
 	)
 	(label "DB PIN 10"
-		(at 284.48 256.54 180)
+		(at 308.61 254 180)
 		(fields_autoplaced yes)
 		(effects
@@
 	)
 	(label "DB PIN 30"
-		(at 284.48 307.34 180)
+		(at 308.61 304.8 180)
 		(fields_autoplaced yes)
 		(effects
@@
 	)
 	(label "DB PIN 7"
-		(at 284.48 248.92 180)
+		(at 308.61 246.38 180)
 		(fields_autoplaced yes)
 		(effects
@@
 	)
 	(label "DB PIN 9"
-		(at 284.48 254 180)
+		(at 308.61 251.46 180)
 		(fields_autoplaced yes)
 		(effects
@@
 	)
 	(label "DB PIN 1"
-		(at 284.48 233.68 180)
+		(at 308.61 231.14 180)
 		(fields_autoplaced yes)
 		(effects
@@
 	)
 	(label "DB PIN 2"
-		(at 284.48 236.22 180)
+		(at 308.61 233.68 180)
 		(fields_autoplaced yes)
 		(effects
@@
 	)
 	(label "DB PIN 15"
-		(at 284.48 269.24 180)
+		(at 308.61 266.7 180)
 		(fields_autoplaced yes)
 		(effects
@@
 	)
 	(label "DB PIN 19"
-		(at 284.48 279.4 180)
+		(at 308.61 276.86 180)
 		(fields_autoplaced yes)
 		(effects
@@
 	)
 	(label "DB PIN 21"
-		(at 284.48 284.48 180)
+		(at 308.61 281.94 180)
 		(fields_autoplaced yes)
 		(effects
@@
 	)
 	(label "DB PIN 4"
-		(at 284.48 241.3 180)
+		(at 308.61 238.76 180)
 		(fields_autoplaced yes)
 		(effects
@@
 	)
 	(label "DB PIN 25"
-		(at 284.48 294.64 180)
+		(at 308.61 292.1 180)
 		(fields_autoplaced yes)
 		(effects
@@
 	)
 	(label "DB PIN 12"
-		(at 284.48 261.62 180)
+		(at 308.61 259.08 180)
 		(fields_autoplaced yes)
 		(effects
@@
 	)
 	(label "DB PIN 29"
-		(at 284.48 304.8 180)
+		(at 308.61 302.26 180)
 		(fields_autoplaced yes)
 		(effects
@@
 	)
 	(label "DB PIN 22"
-		(at 284.48 287.02 180)
+		(at 308.61 284.48 180)
 		(fields_autoplaced yes)
 		(effects
@@
 	)
 	(label "DB PIN 6"
-		(at 284.48 246.38 180)
+		(at 308.61 243.84 180)
 		(fields_autoplaced yes)
 		(effects
@@
 	)
 	(label "DB PIN 16"
-		(at 284.48 271.78 180)
+		(at 308.61 269.24 180)
 		(fields_autoplaced yes)
 		(effects
@@
 	)
 	(label "DB PIN 23"
-		(at 284.48 289.56 180)
+		(at 308.61 287.02 180)
 		(fields_autoplaced yes)
 		(effects
@@
 	)
 	(label "DB PIN 5"
-		(at 284.48 243.84 180)
+		(at 308.61 241.3 180)
 		(fields_autoplaced yes)
 		(effects
@@
 	)
 	(label "DB PIN 17"
-		(at 284.48 274.32 180)
+		(at 308.61 271.78 180)
 		(fields_autoplaced yes)
 		(effects
@@
 	)
 	(label "DB PIN 27"
-		(at 284.48 299.72 180)
+		(at 308.61 297.18 180)
 		(fields_autoplaced yes)
 		(effects
@@
 	)
 	(label "DB PIN 26"
-		(at 284.48 297.18 180)
+		(at 308.61 294.64 180)
 		(fields_autoplaced yes)
 		(effects
@@
 	(symbol
 		(lib_id "Connector_Generic:Conn_01x30")
-		(at 289.56 269.24 0)
+		(at 313.69 266.7 0)
 		(unit 1)
 		(exclude_from_sim no)
@@
 		(dnp no)
 		(property "Reference" "J14"
-			(at 292.1 267.9699 0)
+			(at 316.23 265.4299 0)
 			(effects
 				(font
@@
 		)
 		(property "Value" "Daughter"
-			(at 292.1 270.5099 0)
+			(at 316.23 267.9699 0)
 			(effects
 				(font
@@
 		)
 		(property "Footprint" "AT-Footprints:AMPHENOL_SFV30R-4STE1HLF - FFC - 30 RA"
-			(at 289.56 267.97 0)
+			(at 313.69 265.43 0)
 			(effects
 				(font
@@
 		)
 		(property "Datasheet" "~"
-			(at 289.56 267.97 0)
+			(at 313.69 265.43 0)
 			(effects
 				(font
@@
 		)
 		(property "Description" "Generic connector, single row, 01x30, script generated (kicad-library-utils/schlib/autogen/connector/)"
-			(at 289.56 267.97 0)
+			(at 313.69 265.43 0)
 			(effects
 				(font
@@
 		)
 		(property "Control" ""
-			(at 289.56 267.97 0)
+			(at 313.69 265.43 0)
 			(effects
 				(font
@@
 		)
 		(property "Note" ""
-			(at 289.56 267.97 0)
+			(at 313.69 265.43 0)
 			(effects
 				(font
@@
 		)
 		(property "Sim.Device" ""
-			(at 289.56 267.97 0)
+			(at 313.69 265.43 0)
 			(effects
 				(font
@@
 		)
 		(property "Sim.Pins" ""
-			(at 289.56 267.97 0)
+			(at 313.69 265.43 0)
 			(effects
 				(font
@@
 		)
 		(property "Spec" ""
-			(at 289.56 267.97 0)
+			(at 313.69 265.43 0)
 			(effects
 				(font
@@
 		)
 		(property "LCSC" ""
-			(at 289.56 269.24 0)
+			(at 313.69 266.7 0)
 			(effects
 				(font
@@
 		)
 		(property "MANUFACTURER" ""
-			(at 289.56 269.24 0)
+			(at 313.69 266.7 0)
 			(effects
 				(font
@@
 		)
 		(property "MAXIMUM_PACKAGE_HEIGHT" ""
-			(at 289.56 269.24 0)
+			(at 313.69 266.7 0)
 			(effects
 				(font
@@
 		)
 		(property "PARTREV" ""
-			(at 289.56 269.24 0)
+			(at 313.69 266.7 0)
 			(effects
 				(font
@@
 		)
 		(property "STANDARD" ""
-			(at 289.56 269.24 0)
+			(at 313.69 266.7 0)
 			(effects
 				(font
@@
 		)
 		(instances
-			(project "Occasional Table Too"
+			(project "Superstitious Acrobat"
 				(path "/b48a24c3-e448-4ffe-b89b-bee99abc70c9"
 					(page "5")
@@
 		)
 		(instances
-			(project "Occasional Table Too"
+			(project "Superstitious Acrobat"
 				(path "/b48a24c3-e448-4ffe-b89b-bee99abc70c9"
 					(page "4")
@@
 		)
 		(instances
-			(project "Occasional Table Too"
+			(project "Superstitious Acrobat"
 				(path "/b48a24c3-e448-4ffe-b89b-bee99abc70c9"
 					(page "6")
@@
 		)
 		(instances
-			(project "Occasional Table Too"
+			(project "Superstitious Acrobat"
 				(path "/b48a24c3-e448-4ffe-b89b-bee99abc70c9"
 					(page "2")
@@
 		)
 		(instances
-			(project "Occasional Table Too"
+			(project "Superstitious Acrobat"
 				(path "/b48a24c3-e448-4ffe-b89b-bee99abc70c9"
 					(page "3")
