File: Tools/AT-Interface-Template/AT-Interface-Template.kicad_pcb (KiCad board)
At the start: 2 copper layers, 100 x 94 mm, 16 parts

Commit message: big old push of morphine to commit war crimes
Parts:
- removed H10, H11, H12, H13, H14, H15, H16, H7, H8, H9: Mousebite, mousebites:mouse-bite-2mm-slot
- removed H5, H6: M3, MountingHole:MountingHole_3.2mm_M3_DIN965_Pad
- added FID1: Fiducial, Fiducial:Fiducial_1mm_Mask2mm, F.Cu at (123.4, 45.5)
- added FID2: Fiducial, Fiducial:Fiducial_1mm_Mask2mm, F.Cu at (208.0, 45.5)
- added FID3: Fiducial, Fiducial:Fiducial_1mm_Mask2mm, F.Cu at (123.4, 137.8)
- added FID4: Fiducial, Fiducial:Fiducial_1mm_Mask2mm, F.Cu at (208.0, 137.8)
- added G***: LOGO, AT-Footprints:at-logo, F.Cu at (40.8, 147.3)
- added G***: LOGO, AT-Footprints:at-logo, B.Cu at (170.7, 91.6)
- added J1: IN, AT-Footprints:SJ3-3505, F.Cu at (122.1, 91.6)
- added J11: INT, AT-Footprints:ffc-30-v-TE_3-1734742-0, B.Cu at (165.7, 71.6)
- added J13: INT, AT-Footprints:ffc-30-v-TE_3-1734742-0, B.Cu at (165.7, 81.6)
- added J14: IN, AT-Footprints:SJ3-3505, F.Cu at (120.7, 81.6)
- added J15: IN, AT-Footprints:SJ3-3505, F.Cu at (133.2, 81.6)
- added J16: IN, AT-Footprints:SJ3-3505, F.Cu at (145.7, 81.6)
- added J17: IN, AT-Footprints:SJ3-3505, F.Cu at (185.7, 81.6)
- added J18: IN, AT-Footprints:SJ3-3505, F.Cu at (198.2, 81.6)
- added J19: IN, AT-Footprints:SJ3-3505, F.Cu at (210.7, 81.6)
- added J2: IN, AT-Footprints:SJ3-3505, F.Cu at (134.6, 91.6)
- added J20: INT, AT-Footprints:ffc-30-v-TE_3-1734742-0, B.Cu at (165.7, 61.6)
- added J21: IN, AT-Footprints:SJ3-3505, F.Cu at (185.7, 61.6)
- added J22: IN, AT-Footprints:SJ3-3505, F.Cu at (198.2, 61.6)
- added J23: IN, AT-Footprints:SJ3-3505, F.Cu at (210.7, 61.6)
- added J24: HDMI, AT-Footprints:HDMI-v-PHOENIX_1332073, F.Cu at (128.1, 134.6)
- added J25: 1, AT-Footprints:SJ3-3505, F.Cu at (139.3, 121.7)
- added J26: 2, AT-Footprints:SJ3-3505, F.Cu at (145.5, 131.7)
- added J27: 3, AT-Footprints:SJ3-3505, F.Cu at (151.8, 121.7)
- added J28: 4, AT-Footprints:SJ3-3505, F.Cu at (158.0, 131.7)
- added J29: 5, AT-Footprints:SJ3-3505, F.Cu at (164.3, 121.7)
- added J3: IN, AT-Footprints:SJ3-3505, F.Cu at (147.1, 91.6)
- added J30: 6, AT-Footprints:SJ3-3505, F.Cu at (170.5, 131.7)
- added J31: 7, AT-Footprints:SJ3-3505, F.Cu at (176.8, 121.7)
- added J32: 8, AT-Footprints:SJ3-3505, F.Cu at (183.0, 131.7)
- added J33: 9, AT-Footprints:SJ3-3505, F.Cu at (189.3, 121.7)
- added J34: M, AT-Footprints:SJ3-3505, F.Cu at (195.5, 131.7)
- added J35: INT, AT-Footprints:ffc-30-v-TE_3-1734742-0, B.Cu at (206.4, 126.3)
- added J36: IN, AT-Footprints:SJ3-3505, F.Cu at (122.5, 101.6)
- added J37: LEFT, AT-Footprints:SJ3-3505, F.Cu at (130.0, 111.6)
- added J38: RIGHT, AT-Footprints:SJ3-3505, F.Cu at (135.0, 101.6)
- added J39: IN, AT-Footprints:SJ3-3505, F.Cu at (142.5, 111.6)
- added J4: IN, AT-Footprints:SJ3-3505, F.Cu at (159.6, 91.6)
- added J40: LEFT, AT-Footprints:SJ3-3505, F.Cu at (147.5, 101.6)
- added J41: RIGHT, AT-Footprints:SJ3-3505, F.Cu at (155.0, 111.6)
- added J42: IN, AT-Footprints:SJ3-3505, F.Cu at (160.0, 101.6)
- added J43: LEFT, AT-Footprints:SJ3-3505, F.Cu at (167.5, 111.6)
- added J44: RIGHT, AT-Footprints:SJ3-3505, F.Cu at (172.5, 101.6)
- added J45: IN, AT-Footprints:SJ3-3505, F.Cu at (180.0, 111.6)
- added J46: LEFT, AT-Footprints:SJ3-3505, F.Cu at (185.0, 101.6)
- added J47: RIGHT, AT-Footprints:SJ3-3505, F.Cu at (192.5, 111.6)
- added J48: IN, AT-Footprints:SJ3-3505, F.Cu at (197.5, 101.6)
- added J49: LEFT, AT-Footprints:SJ3-3505, F.Cu at (205.0, 111.6)
- added J5: IN, AT-Footprints:SJ3-3505, F.Cu at (172.1, 91.6)
- added J50: RIGHT, AT-Footprints:SJ3-3505, F.Cu at (210.0, 101.6)
- added J6: IN, AT-Footprints:SJ3-3505, F.Cu at (184.6, 91.6)
- added J7: IN, AT-Footprints:SJ3-3505, F.Cu at (197.1, 91.6)
- added J8: IN, AT-Footprints:SJ3-3505, F.Cu at (209.6, 91.6)
- added JP1: JOIN L, Jumper:SolderJumper-2_P1.3mm_Open_RoundedPad1.0x1.5mm, B.Cu at (158.8, 91.6)
- added JP10: DMONO, Jumper:SolderJumper-2_P1.3mm_Open_RoundedPad1.0x1.5mm, B.Cu at (130.0, 111.6)
- added JP11: DMONO, Jumper:SolderJumper-2_P1.3mm_Open_RoundedPad1.0x1.5mm, B.Cu at (147.5, 101.6)
- added JP12: DMONO, Jumper:SolderJumper-2_P1.3mm_Open_RoundedPad1.0x1.5mm, B.Cu at (155.0, 111.6)
- added JP13: DMONO, Jumper:SolderJumper-2_P1.3mm_Open_RoundedPad1.0x1.5mm, B.Cu at (167.5, 111.6)
- added JP14: DMONO, Jumper:SolderJumper-2_P1.3mm_Open_RoundedPad1.0x1.5mm, B.Cu at (172.5, 101.6)
- added JP15: DMONO, Jumper:SolderJumper-2_P1.3mm_Open_RoundedPad1.0x1.5mm, B.Cu at (185.0, 101.6)
- added JP16: DMONO, Jumper:SolderJumper-2_P1.3mm_Open_RoundedPad1.0x1.5mm, B.Cu at (192.5, 111.6)
- added JP17: DMONO, Jumper:SolderJumper-2_P1.3mm_Open_RoundedPad1.0x1.5mm, B.Cu at (205.0, 111.6)
- added JP18: DMONO, Jumper:SolderJumper-2_P1.3mm_Open_RoundedPad1.0x1.5mm, B.Cu at (210.0, 101.6)
- added JP2: JOIN R, Jumper:SolderJumper-2_P1.3mm_Open_RoundedPad1.0x1.5mm, B.Cu at (171.3, 91.6)
- added JP3: STEREO CONF, Jumper:SolderJumper-3_P1.3mm_Open_Pad1.0x1.5mm_NumberLabels, B.Cu at (122.0, 91.6)
- added JP9: DMONO, Jumper:SolderJumper-2_P1.3mm_Open_RoundedPad1.0x1.5mm, B.Cu at (135.0, 101.6)
- added REF**: OSHW-Logo2_7.3x6mm_SilkScreen, Symbol:OSHW-Logo2_7.3x6mm_SilkScreen, B.Cu at (179.1, 91.6)
- added RV1: PTV09 Pot V, AT-Footprints:2HP_PTV09A-1_Single_Vertical, F.Cu at (127.7, 69.1)
- added RV2: PTV09 Pot V, AT-Footprints:2HP_PTV09A-1_Single_Vertical, F.Cu at (145.7, 69.1)
- added RV3: PTV09 Pot V, AT-Footprints:2HP_PTV09A-1_Single_Vertical, F.Cu at (149.7, 74.1)
- added RV4: PTV09 Pot V, AT-Footprints:2HP_PTV09A-1_Single_Vertical, F.Cu at (181.7, 69.1)
- added RV5: PTV09 Pot V, AT-Footprints:2HP_PTV09A-1_Single_Vertical, F.Cu at (185.7, 74.1)
- added RV6: PTV09 Pot V, AT-Footprints:2HP_PTV09A-1_Single_Vertical, F.Cu at (203.7, 74.1)
- added RV7: PTV09 Pot HZ, AT-Footprints:2HP_PTV09A-1_Single_Vertical, F.Cu at (127.7, 59.1)
- added RV8: PTV09 Pot HZ, AT-Footprints:2HP_PTV09A-1_Single_Vertical, F.Cu at (145.7, 59.1)
- added RV9: PTV09 Pot HZ, AT-Footprints:2HP_PTV09A-1_Single_Vertical, F.Cu at (149.7, 64.1)
- H1, H2, H3, H4: value M3 -> Tooling; footprint MountingHole:MountingHole_3.2mm_M3_DIN965_Pad -> MountingHole:MountingHole_2mm
- moved H3 54.5 mm to (118.2, 139.1)
- moved H4 52.4 mm to (213.2, 139.1)
- moved H1 43.2 mm to (118.2, 44.1)
- moved H2 40.5 mm to (213.2, 44.1)
Routing:
- removed copper zone on B.Cu, net GND
- removed copper zone on F.Cu, net GND
Other:
- board size 100 x 94 mm -> 185 x 128.5 mm
- board text added: "10HP"
- board text added: "2HP"
- board text added: "4HP"
- board text added: "6HP"
- board text added: "8HP"
- board text added: "Deopfer"
- board text added: "PCB Edge"
- board text added: "Short"
- board text added: "V-CUT"
- board text added: "[AUDIO THING NAME]"
- board text removed: "4:3 10DO"
- board text removed: "Butt Why?"
- board text removed: "ONE-8-DM5"
- board text removed: "∅3.2mm {M3}"
