File: Tools/AT-Interface-Template/AT-Interface-Template.kicad_sch (KiCad schematic)
At the start: 2 parts, among them J11 EXT_INTERFACE_1, J14 Daughter

Commit message: big old push of morphine to commit war crimes
Parts:
- removed J11: EXT_INTERFACE_1, AT-Footprints:AMPHENOL_SFV30R-4STE1HLF - FFC - 30 RA, symbol Connector_Generic:Conn_01x30
- removed J14: Daughter, AT-Footprints:AMPHENOL_SFV30R-4STE1HLF - FFC - 30 RA, symbol Connector_Generic:Conn_01x30
- added J10: INT, AT-Footprints:ffc-30-v-TE_3-1734742-0, symbol Connector_Generic:Conn_01x31
- added J12: EXT_INTERFACE_1, AT-Footprints:AMPHENOL_SFV30R-4STE1HLF - FFC - 30 RA, symbol Connector_Generic:Conn_01x30
Connections:
- net +12V: now also J10.1 (Pin_1), J10.2 (Pin_2), J12.1 (Pin_1), J12.2 (Pin_2)
- net -12V: now also J10.29 (Pin_29), J10.30 (Pin_30), J12.29 (Pin_29), J12.30 (Pin_30)
- net EXT_JACK_R_1: now also J12.7 (Pin_7)
- net EXT_JACK_R_2: now also J12.11 (Pin_11)
- net EXT_JACK_R_3: now also J12.14 (Pin_14)
- net EXT_JACK_R_4: now also J12.16 (Pin_16)
- net EXT_JACK_R_5: now also J12.19 (Pin_19)
- net EXT_JACK_R_6: now also J12.21 (Pin_21)
- net EXT_JACK_R_7: now also J12.24 (Pin_24)
- net EXT_JACK_R_8: now also J12.26 (Pin_26)
- net EXT_JACK_TN_1: now also J12.6 (Pin_6)
- net EXT_JACK_TN_2: now also J12.10 (Pin_10)
- net EXT_JACK_T_1: now also J12.5 (Pin_5)
- net EXT_JACK_T_2: now also J12.9 (Pin_9)
- net EXT_JACK_T_3: now also J12.13 (Pin_13)
- net EXT_JACK_T_4: now also J12.15 (Pin_15)
- net EXT_JACK_T_5: now also J12.18 (Pin_18)
- net EXT_JACK_T_6: now also J12.20 (Pin_20)
- net EXT_JACK_T_7: now also J12.23 (Pin_23)
- net EXT_JACK_T_8: now also J12.25 (Pin_25)
- net GND: now also J10.12 (Pin_12), J10.19 (Pin_19), J10.23 (Pin_23), J10.27 (Pin_27), J10.28 (Pin_28), J10.3 (Pin_3), J10.4 (Pin_4), J10.8 (Pin_8), J10.S1, J12.12 (Pin_12), J12.17 (Pin_17), J12.22 (Pin_22), J12.27 (Pin_27), J12.28 (Pin_28), J12.3 (Pin_3), J12.4 (Pin_4), J12.8 (Pin_8)
- new net INT 1 - A: J10.5 (Pin_5)
- new net INT 1 - B: J10.6 (Pin_6)
- new net INT 1 - C: J10.7 (Pin_7)
- new net INT 2 - A: J10.9 (Pin_9)
- new net INT 2 - B: J10.10 (Pin_10)
- new net INT 2 - C: J10.11 (Pin_11)
- new net INT 3 - A: J10.13 (Pin_13)
- new net INT 3 - B: J10.14 (Pin_14)
- new net INT 3 - C: J10.15 (Pin_15)
- new net INT 4 - A: J10.16 (Pin_16)
- new net INT 4 - B: J10.17 (Pin_17)
- new net INT 4 - C: J10.18 (Pin_18)
- new net INT 5 - A: J10.20 (Pin_20)
- new net INT 5 - B: J10.21 (Pin_21)
- new net INT 5 - C: J10.22 (Pin_22)
- new net INT 6 - A: J10.24 (Pin_24)
- new net INT 6 - B: J10.25 (Pin_25)
- new net INT 6 - C: J10.26 (Pin_26)
Other:
- added sheet ExtraMult (extramult.kicad_sch)
- added sheet HDMI (HDMI.kicad_sch)
- added sheet Jacks (jacks.kicad_sch)
- added sheet Pot+Jack (pot+jack.kicad_sch)
- added sheet Pots (pot.kicad_sch)
- added sheet Stereo y (StereoY.kicad_sch)
