File: Tools/AT-Interface-Template/Mechanical.kicad_sch (KiCad schematic)
At the start: 16 parts

Commit message: big old push of morphine to commit war crimes
Parts:
- removed H1, H13, H14, H15, H16, H8: M3, MountingHole:MountingHole_3.2mm_M3_DIN965_Pad, symbol Mechanical:MountingHole_Pad
- removed H10, H11, H12, H5, H6, H7, H9: Mousebite, mousebites:mouse-bite-2mm-slot, symbol Mechanical:MountingHole
- added FID1, FID2, FID3, FID4: Fiducial, Fiducial:Fiducial_1mm_Mask2mm, symbol Mechanical:Fiducial
- added H1: Tooling, MountingHole:MountingHole_2mm, symbol Mechanical:MountingHole
- H2, H3, H4: value Mousebite -> Tooling; footprint mousebites:mouse-bite-2mm-slot -> MountingHole:MountingHole_2mm
