File: Tools/AT-Template/AT-Template.kicad_pcb (KiCad board)
At the start: 2 copper layers, 100 x 100 mm, 31 parts, among them J10 Stereo Jack - SMD HZ, J11 EXT_INTERFACE_1, J14 Daughter, J2 OPT EURO, J4 USB, J5 Audio In, J6 Audio Out, J7 UART, J8 I2C, J9 Stereo Jack - SMD HZ, SW1 Micro Toggle

Commit message: big old push of morphine to commit war crimes
Parts:
- added REF**: MountingHole_3.2mm_M3_DIN965_Pad, MountingHole:MountingHole_3.2mm_M3_DIN965_Pad, F.Cu at (43.2, 200.9)
- moved J11 56.4 mm to (80.9, 81.8)
- moved J14 26.5 mm to (106.9, 118.3)
- moved H2 7.07 mm to (174.8, 95.8)
- moved H1 5.00 mm to (129.8, 95.8)
- moved H4 5.00 mm to (174.8, 140.8)
Routing:
- removed copper zone on F.Cu, net GND
Other:
- board size 100 x 100 mm -> 186.6 x 245 mm
