File: Workshop/PSU/PSU.kicad_pcb (KiCad board)
At the start: 2 copper layers, 100 x 100 mm, 38 parts, among them J10 EURO_CONN, J11 EURO_CONN, J12 EURO_CONN, J2 OPT_DC, J3 EURO_CONN, J4 INT_USB, J5 EURO_CONN, J6 EURO_CONN, J7 EURO_CONN, J8 EURO_CONN, J9 EURO_CONN, Q1 2N3904, U7 STUSB4500QTR, U8 LM2596T-12, U9 LM2596T-12

Commit message: big old push of morphine to commit war crimes
Parts:
- removed D4: SK32, AT-Footprints:M-FLAT_TOS
- removed D6: SK33, AT-Footprints:M-FLAT_TOS
- removed HS1, HS2: HSE-B250-04H, AT-Footprints:HS - LM2596
- removed J10, J12, J5, J6, J7, J8, J9: EURO_CONN, AT-Footprints:EURO_VERT CONN16_S161_OST
- removed J4: INT_USB, Connector_USB:USBC_USBA_2.0_VERT_ADAMTECH_USB-C31-A-D-VT-CS1
- removed L1: 53uH, AT-Footprints:IND_HCTI-68-7.7
- added C10: 100nF, Capacitor_SMD:C_0805_2012Metric_Pad1.18x1.45mm_HandSolder, F.Cu at (71.5, 107.0)
- added C11: 47uf, Capacitor_SMD:C_0805_2012Metric_Pad1.18x1.45mm_HandSolder, F.Cu at (69.5, 95.5)
- added C12: 680nF, Capacitor_SMD:C_0805_2012Metric_Pad1.18x1.45mm_HandSolder, F.Cu at (41.0, 160.6)
- added C13: 56uF, Capacitor_SMD:CP_Elec_6.3x7.7, F.Cu at (44.0, 125.0)
- added C14: 56uF, Capacitor_SMD:CP_Elec_6.3x7.7, F.Cu at (44.3, 142.1)
- added C15: 150pF, Capacitor_SMD:C_0805_2012Metric_Pad1.18x1.45mm_HandSolder, F.Cu at (29.0, 162.6)
- added C16: 100uF, Capacitor_SMD:CP_Elec_8x6.9, F.Cu at (37.5, 133.6)
- added C17: 4.7uf, Capacitor_SMD:C_0805_2012Metric_Pad1.18x1.45mm_HandSolder, F.Cu at (18.5, 153.1)
- added C18: 4.7uf, Capacitor_SMD:C_0805_2012Metric_Pad1.18x1.45mm_HandSolder, F.Cu at (44.2, 147.8)
- added C19: 2.2uf, Capacitor_SMD:C_0805_2012Metric_Pad1.18x1.45mm_HandSolder, F.Cu at (11.7, 99.3)
- added C20: 4.7uf, Capacitor_SMD:C_0805_2012Metric_Pad1.18x1.45mm_HandSolder, F.Cu at (11.7, 102.3)
- added C21: 56uF, Capacitor_SMD:CP_Elec_6.3x7.7, F.Cu at (19.4, 101.9)
- added C22: 56uF, Capacitor_SMD:CP_Elec_6.3x7.7, F.Cu at (19.4, 110.0)
- added C23: 680nF, Capacitor_SMD:C_0805_2012Metric_Pad1.18x1.45mm_HandSolder, F.Cu at (11.7, 105.3)
- added C24: 4.7uf, Capacitor_SMD:C_0805_2012Metric_Pad1.18x1.45mm_HandSolder, F.Cu at (11.7, 108.4)
- added C25: 150pF, Capacitor_SMD:C_0805_2012Metric_Pad1.18x1.45mm_HandSolder, F.Cu at (11.7, 111.4)
- added C26: 100uF, Capacitor_SMD:CP_Elec_8x6.9, F.Cu at (20.5, 119.0)
- added C27: 2.2uf, Capacitor_SMD:C_0805_2012Metric_Pad1.18x1.45mm_HandSolder, F.Cu at (44.2, 162.3)
- added C4: 100nF, Capacitor_SMD:C_0805_2012Metric_Pad1.18x1.45mm_HandSolder, F.Cu at (69.0, 125.4)
- added C5: 10uf, Capacitor_SMD:C_0805_2012Metric_Pad1.18x1.45mm_HandSolder, F.Cu at (63.5, 125.4)
- added C6: 100nF, Capacitor_SMD:C_0805_2012Metric_Pad1.18x1.45mm_HandSolder, F.Cu at (61.5, 125.4)
- added C7: 47uf, Capacitor_SMD:C_0805_2012Metric_Pad1.18x1.45mm_HandSolder, F.Cu at (63.5, 136.9)
- added C8: 100nF, Capacitor_SMD:C_0805_2012Metric_Pad1.18x1.45mm_HandSolder, F.Cu at (64.0, 107.0)
- added C9: 10uf, Capacitor_SMD:C_0805_2012Metric_Pad1.18x1.45mm_HandSolder, F.Cu at (69.5, 107.0)
- added L2: 5.6uH, AT-Footprints:IND_SRP6540-5R6M, F.Cu at (66.5, 100.7)
- added L3: 4.7uH, Inductor_SMD:L_Bourns_SRP5030T, F.Cu at (66.5, 130.7)
- added L4: 56uH, Inductor_THT:L_Radial_D7.8mm_P5.00mm_Fastron_07HCP, F.Cu at (1.96, 102.7)
- added L5: 56uH, Inductor_THT:L_Radial_D7.8mm_P5.00mm_Fastron_07HCP, F.Cu at (36.2, 152.8)
- added R10: 100k, Resistor_SMD:R_0805_2012Metric_Pad1.20x1.40mm_HandSolder, F.Cu at (11.7, 117.4)
- added R11: 1M, Resistor_SMD:R_0805_2012Metric_Pad1.20x1.40mm_HandSolder, F.Cu at (11.7, 120.3)
- added R12: 92k, Resistor_SMD:R_0805_2012Metric_Pad1.20x1.40mm_HandSolder, F.Cu at (11.7, 123.3)
- added R3: 52k3, Resistor_SMD:R_0805_2012Metric_Pad1.20x1.40mm_HandSolder, F.Cu at (62.0, 111.0)
- added R4: 10k, Resistor_SMD:R_0805_2012Metric_Pad1.20x1.40mm_HandSolder, F.Cu at (64.0, 111.0)
- added R5: 140k, Resistor_SMD:R_0805_2012Metric_Pad1.20x1.40mm_HandSolder, F.Cu at (71.0, 121.5)
- added R6: 10k, Resistor_SMD:R_0805_2012Metric_Pad1.20x1.40mm_HandSolder, F.Cu at (69.0, 121.5)
- added R7: 1M, Resistor_SMD:R_0805_2012Metric_Pad1.20x1.40mm_HandSolder, F.Cu at (27.0, 162.6)
- added R8: 100k, Resistor_SMD:R_0805_2012Metric_Pad1.20x1.40mm_HandSolder, F.Cu at (28.8, 150.4)
- added R9: 92k, Resistor_SMD:R_0805_2012Metric_Pad1.20x1.40mm_HandSolder, F.Cu at (23.3, 143.9)
- added U1: LM43601PWPR, Package_SO:HTSSOP-16-1EP_4.4x5mm_P0.65mm_EP3.4x5mm_Mask2.46x2.31mm_ThermalVias, F.Cu at (46.2, 155.5)
- added U2: LM43601PWPR, Package_SO:HTSSOP-16-1EP_4.4x5mm_P0.65mm_EP3.4x5mm_Mask2.46x2.31mm_ThermalVias, F.Cu at (4.37, 120.6)
- added U3: TPS563300, Package_TO_SOT_SMD:SOT-583-8, F.Cu at (66.2, 125.0)
- added U4: TPS563300, Package_TO_SOT_SMD:SOT-583-8, F.Cu at (66.7, 107.5)
- D5, R1, R13, R17, R18, R2: moved to F.Cu
- moved D7 165.4 mm to (102.1, 116.3), turned to 0 degrees
- moved D1 164.3 mm to (102.1, 110.2), turned to 0 degrees
- moved D3 161.9 mm to (102.1, 113.2), turned to 0 degrees
- moved R13 146.6 mm to (125.5, 114.5), turned to 0 degrees
- moved J3 141.6 mm to (118.4, 87.7), turned to 0 degrees
- moved R1 141.4 mm to (125.5, 108.5), turned to 0 degrees
- moved R2 141.2 mm to (125.5, 111.5), turned to 0 degrees
- moved H7 126.4 mm to (146.0, 102.1), turned to 0 degrees
- moved U9 123.8 mm to (114.0, 126.7), turned to 0 degrees
- moved Q1 120.6 mm to (101.8, 125.6), turned to 0 degrees
- moved C3 118.8 mm to (103.3, 102.9)
- moved D5 117.7 mm to (103.9, 120.0), turned to 0 degrees
- moved H5 110.0 mm to (146.0, 86.1), turned to 0 degrees
- moved U7 108.6 mm to (107.4, 111.9), turned to 0 degrees
- moved R16 104.3 mm to (125.5, 117.4)
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Connections:
- net +12V renamed +12v
- net GND renamed COM
Routing:
- net +12v: track 236.6 -> 24.0 mm, vias 0 -> 2
- net -12V: track 196.5 -> 0.00 mm
- net +5V: track 95.0 -> 0.00 mm
- net /+20V: track 77.5 -> 0.00 mm
- net Net-(D6-K): track 30.9 -> 0.00 mm
- net +5v: track 0.00 -> 24.0 mm, vias 0 -> 2
- net Net-(D4-K): track 23.9 -> 0.00 mm
- net Net-(Q1-C): track 13.1 -> 0.00 mm
- net Net-(D5-A): track 6.72 -> 0.00 mm
- net Net-(U1-CBOOT): track 0.00 -> 5.20 mm
- net PD +15v: track 0.00 -> 4.68 mm
- net Net-(U1-VCC): track 0.00 -> 3.64 mm
- net /12v SW: track 0.00 -> 3.62 mm
- net /5v SW: track 0.00 -> 3.62 mm
- net COM: track 3.40 -> 0.00 mm
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- added copper zone on B.Cu, net -12v B
- added copper zone on F.Cu, net -12v B
- added copper zone on F.Cu, net /-12v B CBOOT
- added copper zone on F.Cu, net /12v FB
- added copper zone on F.Cu, net /12v SW
- added copper zone on F.Cu, net COM
- added copper zone on F.Cu, net PD +15v
Other:
- board size 100 x 100 mm -> 45 x 85 mm
- board text added: "Regulated +12V"
- board text added: "Regulated +5V"
- board text removed: "HEATSINK IS -12V TO GND"
