File: Workshop/PSU/PSU.kicad_sch (KiCad schematic)
At the start: 41 parts, among them J1 EXT USB C, J10 EURO_CONN, J11 EURO_CONN, J12 EURO_CONN, J2 OPT_DC, J3 EURO_CONN, J4 INT_USB, J5 EURO_CONN, J6 EURO_CONN, J7 EURO_CONN, J8 EURO_CONN, J9 EURO_CONN, Q1 2N3904, U1 DKA30A-12, U2 STUSB4761QTR, U7 STUSB4500QTR, U8 LM2596T-12, U9 LM2596T-12

Commit message: big old push of morphine to commit war crimes
Parts:
- removed U1: DKA30A-12, AT-Footprints:DKA30_MWU, symbol AT-Symbols:DKA30A-12
- removed U2: STUSB4761QTR, AT-Footprints:QFN16_STUSB4761QTR_STM, symbol AT-Symbols:STUSB4761QTR
- added C10, C4, C6, C8: 100nF, Capacitor_SMD:C_0805_2012Metric_Pad1.18x1.45mm_HandSolder, symbol Device:C
- added C11, C7: 47uf, Capacitor_SMD:C_0805_2012Metric_Pad1.18x1.45mm_HandSolder, symbol Device:C
- added C12, C23: 680nF, Capacitor_SMD:C_0805_2012Metric_Pad1.18x1.45mm_HandSolder, symbol Device:C
- added C13, C14, C21, C22: 56uF, Capacitor_SMD:CP_Elec_6.3x7.7, symbol Device:C_Polarized
- added C15, C25: 150pF, Capacitor_SMD:C_0805_2012Metric_Pad1.18x1.45mm_HandSolder, symbol Device:C
- added C16, C26: 100uF, Capacitor_SMD:CP_Elec_8x6.9, symbol Device:C_Polarized
- added C17, C18, C20, C24: 4.7uf, Capacitor_SMD:C_0805_2012Metric_Pad1.18x1.45mm_HandSolder, symbol Device:C
- added C19, C27: 2.2uf, Capacitor_SMD:C_0805_2012Metric_Pad1.18x1.45mm_HandSolder, symbol Device:C
- added C5, C9: 10uf, Capacitor_SMD:C_0805_2012Metric_Pad1.18x1.45mm_HandSolder, symbol Device:C
- added L2: 5.6uH, AT-Footprints:IND_SRP6540-5R6M, symbol Device:L
- added L3: 4.7uH, Inductor_SMD:L_Bourns_SRP5030T, symbol Device:L
- added L4, L5: 56uH, Inductor_THT:L_Radial_D7.8mm_P5.00mm_Fastron_07HCP, symbol Device:L
- added R10, R8: 100k, Resistor_SMD:R_0805_2012Metric_Pad1.20x1.40mm_HandSolder, symbol Device:R
- added R11, R7: 1M, Resistor_SMD:R_0805_2012Metric_Pad1.20x1.40mm_HandSolder, symbol Device:R
- added R12, R9: 92k, Resistor_SMD:R_0805_2012Metric_Pad1.20x1.40mm_HandSolder, symbol Device:R
- added R3: 52k3, Resistor_SMD:R_0805_2012Metric_Pad1.20x1.40mm_HandSolder, symbol Device:R
- added R4, R6: 10k, Resistor_SMD:R_0805_2012Metric_Pad1.20x1.40mm_HandSolder, symbol Device:R
- added R5: 140k, Resistor_SMD:R_0805_2012Metric_Pad1.20x1.40mm_HandSolder, symbol Device:R
- added U1, U2: LM43601PWPR, Package_SO:HTSSOP-16-1EP_4.4x5mm_P0.65mm_EP3.4x5mm_Mask2.46x2.31mm_ThermalVias, symbol AT-Symbols:LM43601PWPR
- added U3, U4: TPS563300, Package_TO_SOT_SMD:SOT-583-8, symbol Regulator_Switching:TPS563300
Connections:
- net +12V: now also C7.2, L3.2, R5.2
- net GND: now also C10.2, C11.1, C13.2, C14.2, C15.1, C16.1, C17.1, C19.2, C20.2, C21.2, C22.2, C24.1, C24.2, C25.1, C25.2, C26.1, C26.2, C5.2, C6.2, C7.1, C9.2, L4.2, L5.2, R10.1, R11.1, R11.2, R12.1, R12.2, R4.2, R6.2, R7.1, R8.1, U1.5 (BIAS), U2.10 (AGND), U2.15 (PGND), U2.16 (PGND), U2.5 (BIAS), U2.PAD, U3.4 (GND), U4.4 (GND)
- new net: C23.1, L4.1, U2.1 (SW), U2.2 (SW)
- new net: C23.2, U2.3 (CBOOT)
- new net: C19.1, U2.4 (VCC)
- new net: R10.2, U2.8 (PGOOD)
- new net: C8.2, U4.6 (BST)
- new net: C4.2, U3.6 (BST)
- new net: R8.2, U1.8 (PGOOD)
- new net: C12.2, U1.3 (CBOOT)
- new net: C27.1, U1.4 (VCC)
- new net +5v: C11.2, L2.2, R3.2
- new net -12v B: C16.2, C17.2, C18.2, C27.2, R9.2, U1.10 (AGND), U1.15 (PGND), U1.16 (PGND), U1.PAD
- new net -12v B Bias: C15.2, R7.2, R9.1, U1.9 (FB)
- new net -12v B CBOOT: C12.1, L5.1, U1.1 (SW), U1.2 (SW)
- new net 12v FB: R5.1, R6.1, U3.8 (FB)
- new net 12v SW: C4.1, L3.1, U3.5 (SW)
- new net 5v FB: R3.1, R4.1, U4.8 (FB)
- new net 5v SW: C8.1, L2.1, U4.5 (SW)
- new net PD +15v: C10.1, C13.1, C14.1, C18.1, C20.1, C21.1, C22.1, C5.1, C6.1, C9.1, U1.12 (EN), U1.13 (VIN), U1.14 (VIN), U2.12 (EN), U2.13 (VIN), U2.14 (VIN), U3.3 (VIN), U4.3 (VIN)
- no-connect marks 8 -> 16
Other:
- added sheet USBC (PD.kicad_sch)
- note added: "Regulated -12v/1A"
- note added: "Regulated 12v/2A"
- note added: "Regulated 5v/2A"
