File: Workshop/DEitW/DEitW.kicad_pcb (KiCad board)
At the start: 2 copper layers, 183.5 x 130.8 mm, 109 parts, among them J11 EXT_INTERFACE_1, J12 Stereo Jack - SMD HZ, J13 Stereo Jack - SMD HZ, J14 Daughter, J15 Stereo Jack - SMD HZ, J16 Stereo Jack - SMD HZ, J17 Stereo Jack - SMD HZ, J18 Stereo Jack - SMD HZ, J19 Stereo Jack - SMD HZ, J2 OPT EURO, J20 Stereo Jack - SMD HZ, J21 Stereo Jack - SMD HZ, J22 Stereo Jack - SMD HZ, J23 Stereo Jack - SMD HZ, J24 Stereo Jack - SMD HZ, J4 USB, J5 Audio In, J6 Audio Out, J7 UART, J8 I2C, J9 AudioJack3_SwitchT, Q1 BC847BDW1, Q2 BC847BDW1, Q3 BC847BDW1, Q4 BC847BDW1, Q5 BC847BDW1, Q6 BC847BDW1, Q7 BC847BDW1, Q8 BC847BDW1, Q9 BC847BDW1, U1 TLC555xD, U3 TLC555xD, U5 TLC555xD, U6 TLC555xD, U8 TLC555xD, U9 TLC555xD

Commit message: polished and PSU, did a todo, much ado about something
Parts:
- moved J9 162.1 mm to (209.4, 160.1)
- moved REF** 162.1 mm to (128.3, 158.1)
- moved REF** 162.1 mm to (125.9, 155.7)
Other:
- board size 183.5 x 130.8 mm -> 100.3 x 113.3 mm
Changed lines of the file:
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@@
 		(tags "SOD-323")
 		(property "Reference" "D19"
-			(at 0 -1.850001 360)
+			(at 0 -1.850001 0)
 			(layer "F.SilkS")
 			(effects
@@
 		(tags "LED")
 		(property "Reference" "D26"
-			(at 0 -1.65 360)
+			(at 0 -1.65 0)
 			(layer "F.SilkS")
 			(effects
@@
 		(tags "SOT-363 SC-70-6 SC-88")
 		(property "Reference" "Q6"
-			(at 0 -2.25 360)
+			(at 0 -2.25 0)
 			(layer "F.SilkS")
 			(effects
@@
 		(tags "SOD-323")
 		(property "Reference" "D20"
-			(at 0 -1.850001 360)
+			(at 0 -1.850001 0)
 			(layer "F.SilkS")
 			(effects
@@
 		(tags "SOD-323")
 		(property "Reference" "D17"
-			(at 0 -1.850001 360)
+			(at 0 -1.850001 0)
 			(layer "F.SilkS")
 			(effects
@@
 		(tags "SOD-323")
 		(property "Reference" "D24"
-			(at 0 -1.850001 360)
+			(at 0 -1.850001 0)
 			(layer "F.SilkS")
 			(effects
@@
 	(footprint "Fiducial:Fiducial_1mm_Mask3mm"
 		(layer "F.Cu")
-		(at 45.1125 18.9)
+		(at 128.2625 158.05)
 		(descr "Circular Fiducial, 1mm bare copper, 3mm soldermask opening (recommended)")
 		(tags "fiducial")
@@
 		(tags "SOD-323")
 		(property "Reference" "D33"
-			(at 0 -1.850001 360)
+			(at 0 -1.850001 0)
 			(layer "F.SilkS")
 			(effects
@@
 		(tags "SOD-323")
 		(property "Reference" "D22"
-			(at 0 -1.850001 360)
+			(at 0 -1.850001 0)
 			(layer "F.SilkS")
 			(effects
@@
 		(tags "SOD-323")
 		(property "Reference" "D21"
-			(at 0 -1.850001 360)
+			(at 0 -1.850001 0)
 			(layer "F.SilkS")
 			(effects
@@
 		(tags "SOD-323")
 		(property "Reference" "D27"
-			(at 0 -1.850001 360)
+			(at 0 -1.850001 0)
 			(layer "F.SilkS")
 			(effects
@@
 		(tags "SOD-323")
 		(property "Reference" "D32"
-			(at 0 -1.850001 360)
+			(at 0 -1.850001 0)
 			(layer "F.SilkS")
 			(effects
@@
 		(tags "SOD-323")
 		(property "Reference" "D23"
-			(at 0 -1.850001 360)
+			(at 0 -1.850001 0)
 			(layer "F.SilkS")
 			(effects
@@
 		(tags "LED")
 		(property "Reference" "D25"
-			(at 0 -1.65 360)
+			(at 0 -1.65 0)
 			(layer "F.SilkS")
 			(effects
@@
 		(tags "SOD-323")
 		(property "Reference" "D34"
-			(at 0 -1.850001 360)
+			(at 0 -1.850001 0)
 			(layer "F.SilkS")
 			(effects
@@
 		(tags "SOIC SO")
 		(property "Reference" "U8"
-			(at 0 -3.4 360)
+			(at 0 -3.4 0)
 			(layer "F.SilkS")
 			(effects
@@
 		(tags "SOIC SO")
 		(property "Reference" "U5"
-			(at 0 -3.4 360)
+			(at 0 -3.4 0)
 			(layer "F.SilkS")
 			(effects
@@
 		(tags "SOD-323")
 		(property "Reference" "D31"
-			(at 0 -1.850001 360)
+			(at 0 -1.850001 0)
 			(layer "F.SilkS")
 			(effects
@@
 		(tags "LED")
 		(property "Reference" "D15"
-			(at 0 -1.65 360)
+			(at 0 -1.65 0)
 			(layer "F.SilkS")
 			(effects
@@
 		(tags "SOT-363 SC-70-6 SC-88")
 		(property "Reference" "Q7"
-			(at 0 -2.25 360)
+			(at 0 -2.25 0)
 			(layer "F.SilkS")
 			(effects
@@
 		(tags "SOT-363 SC-70-6 SC-88")
 		(property "Reference" "Q8"
-			(at 0 -2.25 360)
+			(at 0 -2.25 0)
 			(layer "F.SilkS")
 			(effects
@@
 		(tags "SOD-323")
 		(property "Reference" "D18"
-			(at 0 -1.850001 360)
+			(at 0 -1.850001 0)
 			(layer "F.SilkS")
 			(effects
@@
 		(tags "SOIC SO")
 		(property "Reference" "U9"
-			(at 0 -3.4 360)
+			(at 0 -3.4 0)
 			(layer "F.SilkS")
 			(effects
@@
 	(footprint "AT-Footprints:SJ3"
 		(layer "F.Cu")
-		(at 126.2625 20.9375 90)
+		(at 209.4125 160.0875 90)
 		(property "Reference" "J9"
 			(at -2 -6 90)
@@
 		(tags "SOT-363 SC-70-6 SC-88")
 		(property "Reference" "Q4"
-			(at 0 -2.25 360)
+			(at 0 -2.25 0)
 			(layer "F.SilkS")
 			(effects
@@
 		(tags "SOT-363 SC-70-6 SC-88")
 		(property "Reference" "Q9"
-			(at 0 -2.25 360)
+			(at 0 -2.25 0)
 			(layer "F.SilkS")
 			(effects
@@
 		(tags "SOT-363 SC-70-6 SC-88")
 		(property "Reference" "Q5"
-			(at 0 -2.25 360)
+			(at 0 -2.25 0)
 			(layer "F.SilkS")
 			(effects
@@
 		(tags "SOIC SO")
 		(property "Reference" "U6"
-			(at 0 -3.4 360)
+			(at 0 -3.4 0)
 			(layer "F.SilkS")
 			(effects
@@
 		(tags "SOD-323")
 		(property "Reference" "D29"
-			(at 0 -1.850001 360)
+			(at 0 -1.850001 0)
 			(layer "F.SilkS")
 			(effects
@@
 		(tags "SOD-323")
 		(property "Reference" "D28"
-			(at 0 -1.850001 360)
+			(at 0 -1.850001 0)
 			(layer "F.SilkS")
 			(effects
@@
 	(footprint "MountingHole:MountingHole_2mm"
 		(layer "F.Cu")
-		(at 42.7625 16.55)
+		(at 125.9125 155.7)
 		(descr "Mounting Hole 2mm, no annular")
 		(tags "mounting hole 2mm no annular")
@@
 		(tags "SOD-323")
 		(property "Reference" "D30"
-			(at 0 -1.850001 360)
+			(at 0 -1.850001 0)
 			(layer "F.SilkS")
 			(effects
@@
 		(tags "LED")
 		(property "Reference" "D16"
-			(at 0 -1.65 360)
+			(at 0 -1.65 0)
 			(layer "F.SilkS")
 			(effects
@@
 	)
 	(gr_rect
-		(start 41.2625 15.05)
-		(end 141.2625 20.05)
+		(start 124.4125 154.2)
+		(end 224.4125 159.2)
 		(stroke
 			(width 0.1)
