File: Workshop/EurorATX/EurorATX.kicad_sch (KiCad schematic)
At the start: 31 parts, among them J1 FRONT PANEL MAGIC, J16 MAINBOARD MAGIC, J2 Stereo Jack - SMD HZ, J3 EXT_INTERFACE_1, J4 Daughter, J5 Stereo Jack - SMD HZ, SW1 Micro Toggle, U1 TPS560430XDBVR

Commit message: polished and PSU, did a todo, much ado about something
Other:
- added sheet HDMI (HDMI.kicad_sch)
