File: Workshop/Zoetrope/Zoetrope.kicad_pcb (KiCad board)
At the start: 2 copper layers, 135.2 x 128.5 mm, 134 parts, among them J2 OPT EURO, J38 1/2 Trigger, J39 1/4 Trigger, J4 Bar End Trigger, J40 1/8 Trigger, J41 1/16 Trigger, J42 1/2 Front Gate, J43 1/4 Front Gate, J44 1/8 Front Gate, J45 1/16 Front Gate, J46 1/2 Back Gate, J47 1/4 Back Gate, J48 1/8 Back Gate, J49 1/16 Back Gate, J5 Beat Clock Out, J6 Phrase End Trigger, J7 Gate In - Bank A, Q1 MMBT2222A, SW19 Bar Length _{Coarse}, SW20 Bar Length _{Cont}, SW21 BPM _{Coarse}, SW23 Bar Length _{Cont}, SW24 Bar Length _{Cont}, SW25 Bar Length _{Cont}, SW32 BPM Range, SW33 Phrase Length, SW36 Single Bar, U15 NEX 74HC393BQ,115, U16 40106, U19 74HC08, U20 4017, U21 4017, U22 74LVC1G3157, U23 74LVC1G3157, U24 74LVC1G3157, U25 74LVC1G3157, U26 74LVC1G3157, U27 74LVC1G3157, U28 74LVC1G3157, U29 74LVC1G3157, U30 TL074, U31 TL074, U32 74LVC1G3157, U34 NEX 74HC393BQ,115, U35 NEX 74HC393BQ,115, U36 4017, U37 74HC08, U38 4017, U39 4017, U41 40110, U42 40110, U43 40110, U44 4017, U45 74LVC1G3157, U46 74LVC1G3157, U47 74LVC1G3157, U48 74LVC1G3157, U49 4017, U50 74HC08

Commit message: polished and PSU, did a todo, much ado about something
Parts:
- removed REF**: Valve_ECC-83-1, Valve:Valve_ECC-83-1
Changed lines of the file:
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@@
 		(tags "resistor handsolder")
 		(property "Reference" "R95"
-			(at -4 0 360)
+			(at -4 0 0)
 			(layer "F.SilkS")
 			(effects
@@
 		(tags "resistor handsolder")
 		(property "Reference" "R90"
-			(at -4 0 360)
+			(at -4 0 0)
 			(layer "F.SilkS")
 			(effects
@@
 		(tags "THT DIP DIL PDIP 2.54mm 7.62mm 300mil Socket")
 		(property "Reference" "U41"
-			(at 3.81 -2.33 360)
+			(at 3.81 -2.33 0)
 			(layer "F.SilkS")
 			(effects
@@
 		(tags "resistor handsolder")
 		(property "Reference" "R93"
-			(at -4 0 360)
+			(at -4 0 0)
 			(layer "F.SilkS")
 			(effects
@@
 		(tags "capacitor handsolder")
 		(property "Reference" "C17"
-			(at -4 -0.03 360)
+			(at -4 -0.03 0)
 			(layer "F.SilkS")
 			(effects
@@
 		(tags "resistor handsolder")
 		(property "Reference" "R89"
-			(at 0 2 360)
+			(at 0 2 0)
 			(layer "F.SilkS")
 			(effects
@@
 		)
 	)
-	(footprint "Valve:Valve_ECC-83-1"
-		(layer "F.Cu")
-		(at 85.0625 102.09)
-		(descr "Valve ECC-83-1 round pins")
-		(tags "Valve ECC-83-1 round pins")
-		(property "Reference" "REF**"
-			(at -3.45 -16 0)
-			(layer "F.SilkS")
-			(effects
-				(font
-					(size 1 1)
-					(thickness 0.1)
-				)
-			)
-		)
-		(property "Value" "Valve_ECC-83-1"
-			(at -3.45 6.68 0)
-			(unlocked yes)
-			(layer "F.Fab")
-			(effects
-				(font
-					(size 1 1)
-					(thickness 0.15)
-					(italic yes)
-				)
-			)
-		)
-		(property "Footprint" "Valve:Valve_ECC-83-1"
-			(at 0 0 0)
-			(unlocked yes)
-			(layer "F.Fab")
-			(hide yes)
-			(effects
-				(font
-					(size 1 1)
-					(thickness 0.15)
-					(italic yes)
-				)
-			)
-		)
-		(property "Datasheet" ""
-			(at 0 0 0)
-			(unlocked yes)
-			(layer "F.Fab")
-			(hide yes)
-			(effects
-				(font
-					(size 1 1)
-					(thickness 0.15)
-					(italic yes)
-				)
-			)
-		)
-		(property "Description" ""
-			(at 0 0 0)
-			(unlocked yes)
-			(layer "F.Fab")
-			(hide yes)
-			(effects
-				(font
-					(size 1 1)
-					(thickness 0.15)
-					(italic yes)
-				)
-			)
-		)
-		(attr through_hole)
-		(fp_circle
-			(center -3.45 -4.75)
-			(end 6.71 -3.48)
-			(stroke
-				(width 0.1)
-				(type solid)
-			)
-			(fill none)
-			(layer "F.SilkS")
-		)
-		(fp_circle
-			(center -3.45 -4.75)
-			(end -3.45 -15)
-			(stroke
-				(width 0.05)
-				(type solid)
-			)
-			(fill none)
-			(layer "F.CrtYd")
-		)
-		(fp_circle
-			(center -3.45 -4.75)
-			(end -3.45 -14.75)
-			(stroke
-				(width 0.1)
-				(type solid)
-			)
-			(fill none)
-			(layer "F.Fab")
-		)
-		(fp_text user "${REFERENCE}"
-			(at -3.45 -4.75 0)
-			(unlocked yes)
-			(layer "F.Fab")
-			(effects
-				(font
-					(size 1 1)
-					(thickness 0.15)
-					(italic yes)
-				)
-			)
-		)
-		(pad "1" thru_hole circle
-			(at 0 0)
-			(size 2.03 2.03)
-			(drill 1.02)
-			(layers "*.Cu" "*.Mask")
-			(remove_unused_layers no)
-		)
-		(pad "2" thru_hole circle
-			(at 2.15 -2.93)
-			(size 2.03 2.03)
-			(drill 1.02)
-			(layers "*.Cu" "*.Mask")
-			(remove_unused_layers no)
-		)
-		(pad "3" thru_hole circle
-			(at 2.15 -6.58)
-			(size 2.03 2.03)
-			(drill 1.02)
-			(layers "*.Cu" "*.Mask")
-			(remove_unused_layers no)
-		)
-		(pad "4" thru_hole circle
-			(at 0 -9.51)
-			(size 2.03 2.03)
-			(drill 1.02)
-			(layers "*.Cu" "*.Mask")
-			(remove_unused_layers no)
-		)
-		(pad "5" thru_hole circle
-			(at -3.45 -10.65)
-			(size 2.03 2.03)
-			(drill 1.02)
-			(layers "*.Cu" "*.Mask")
-			(remove_unused_layers no)
-		)
-		(pad "6" thru_hole circle
-			(at -6.91 -9.51)
-			(size 2.03 2.03)
-			(drill 1.02)
-			(layers "*.Cu" "*.Mask")
-			(remove_unused_layers no)
-		)
-		(pad "7" thru_hole circle
-			(at -9.06 -6.58)
-			(size 2.03 2.03)
-			(drill 1.02)
-			(layers "*.Cu" "*.Mask")
-			(remove_unused_layers no)
-		)
-		(pad "8" thru_hole circle
-			(at -9.06 -2.97)
-			(size 2.03 2.03)
-			(drill 1.02)
-			(layers "*.Cu" "*.Mask")
-			(remove_unused_layers no)
-		)
-		(pad "9" thru_hole circle
-			(at -6.91 0)
-			(size 2.03 2.03)
-			(drill 1.02)
-			(layers "*.Cu" "*.Mask")
-			(remove_unused_layers no)
-		)
-		(model "${AT_PROJECT_ROOT}/res/3dmodels/12AX7--3DModel-STEP-1.STEP"
-			(offset
-				(xyz -3.5 5 0)
-			)
-			(scale
-				(xyz 1 1 1)
-			)
-			(rotate
-				(xyz -90 0 0)
-			)
-		)
-	)
 	(footprint "AT-Footprints:TG-3541CE"
 		(layer "F.Cu")
 		(at 161.412501 86.0225)
 		(property "Reference" "X1"
-			(at 0 -0.499999 360)
+			(at 0 -0.499999 0)
 			(layer "F.SilkS")
 			(effects
@@
 		(tags "resistor handsolder")
 		(property "Reference" "R94"
-			(at 0 -2 360)
+			(at 0 -2 0)
 			(layer "F.SilkS")
 			(effects
@@
 		(tags "resistor handsolder")
 		(property "Reference" "R98"
-			(at -4 0 360)
+			(at -4 0 0)
 			(layer "F.SilkS")
 			(effects
@@
 		(tags "capacitor handsolder")
 		(property "Reference" "C18"
-			(at -4 -0.03 360)
+			(at -4 -0.03 0)
 			(layer "F.SilkS")
 			(effects
@@
 		(tags "THT DIP DIL PDIP 2.54mm 7.62mm 300mil Socket")
 		(property "Reference" "U43"
-			(at 3.81 -2.33 360)
+			(at 3.81 -2.33 0)
 			(layer "F.SilkS")
 			(effects
@@
 		(tags "resistor handsolder")
 		(property "Reference" "R82"
-			(at 0 -2.05 360)
+			(at 0 -2.05 0)
 			(layer "B.SilkS")
 			(effects
@@
 		(tags "resistor handsolder")
 		(property "Reference" "R86"
-			(at 0 -1.47 360)
+			(at 0 -1.47 0)
 			(layer "B.SilkS")
 			(effects
@@
 		(tags "resistor handsolder")
 		(property "Reference" "R97"
-			(at 0 -2.000001 360)
+			(at 0 -2.000001 0)
 			(layer "B.SilkS")
 			(effects
@@
 		(tags "resistor handsolder")
 		(property "Reference" "R81"
-			(at 0 2 360)
+			(at 0 2 0)
 			(layer "B.SilkS")
 			(effects
@@
 		(tags "resistor handsolder")
 		(property "Reference" "R87"
-			(at 0 2 360)
+			(at 0 2 0)
 			(layer "B.SilkS")
 			(effects
@@
 		(tags "resistor handsolder")
 		(property "Reference" "R96"
-			(at 0 1.65 360)
+			(at 0 1.65 0)
 			(layer "B.SilkS")
 			(effects
